File: electronique/camion-grue.brd (EAGLE design)
At the start: 160 x 100 mm, 78 parts, among them P1 RGEF800, Q1 BSS138, Q2 BSS138

Commit message: Elec: schéma presque ok + placement des composants
Parts:
- removed ALIM-GRUE: JST-02VL-V, con-jst:VL-02-V
- removed FEUX_ARRIERE: JST-06, con-jst:GH-06-V
- removed H-BRIDGE1:C1, H-BRIDGE1:C2, H-BRIDGE2:C1, H-BRIDGE2:C2, H-BRIDGE3:C1, H-BRIDGE3:C2, H-BRIDGE4:C1, H-BRIDGE4:C2: (no value), resistor:C0805
- removed H-BRIDGE1:D1, H-BRIDGE1:D2, H-BRIDGE1:D3, H-BRIDGE1:D4, H-BRIDGE2:D1, H-BRIDGE2:D2, H-BRIDGE2:D3, H-BRIDGE2:D4, H-BRIDGE3:D1, H-BRIDGE3:D2, H-BRIDGE3:D3, H-BRIDGE3:D4, H-BRIDGE4:D1, H-BRIDGE4:D2, H-BRIDGE4:D3, H-BRIDGE4:D4: 1N4942, diode:DO41-10
- removed H-BRIDGE1:IC1, H-BRIDGE2:IC1, H-BRIDGE3:IC1, H-BRIDGE4:IC1: L298, st-microelectronics:MULTIWATT-15
- removed H-BRIDGE1:R1, H-BRIDGE1:R2, H-BRIDGE1:R3, H-BRIDGE2:R1, H-BRIDGE2:R2, H-BRIDGE2:R3, H-BRIDGE3:R1, H-BRIDGE3:R2, H-BRIDGE3:R3, H-BRIDGE4:R1, H-BRIDGE4:R2, H-BRIDGE4:R3: 10k, resistor:R0805
- removed LIPO-ET-ARRET-URGENCE: JST-04VL-V, con-jst:VL-04-V
- removed SERIAL_GRUE: JST-02GH-V, con-jst:GH-02-V
- removed TOF_FLAN_AV_D, TOF_FLAN_AV_G: JST-05, con-jst:GH-05-V
- removed U$1: TEENSY_3.1-3.2_DIL, Teensy_libSG:TEENSY_3.0-3.2&LC_DIL
- added ARRET_URGENCE, LIPO: JST-12, con-jst:GH-12-V
- added AX12_D, AX12_G: DYNAMIXEL-1X03AX, 1NTech_pinhead:DYNAMIXEL_AX_1X03
- added C10: (no value), 1NTech_RLCD:TT5D11L
- added C5, C6, C7, C8: 1µF, resistor:E2,5-6
- added DELS_ET_TOF_AR: JST-15, con-jst:GH-15-V
- added DEL_GYRO: JST-05, con-jst:GH-05-V
- added GRUE, PHARES_ET_TOF_AV: JST-10, con-jst:GH-10-V
- added H-BRIDGE_AR_D:C1, H-BRIDGE_AR_D:C2, H-BRIDGE_AR_G:C1, H-BRIDGE_AR_G:C2, H-BRIDGE_AV_D:C1, H-BRIDGE_AV_D:C2, H-BRIDGE_AV_G:C1, H-BRIDGE_AV_G:C2: (no value), resistor:C0805
- added H-BRIDGE_AR_D:D1, H-BRIDGE_AR_D:D2, H-BRIDGE_AR_D:D3, H-BRIDGE_AR_D:D4, H-BRIDGE_AR_G:D1, H-BRIDGE_AR_G:D2, H-BRIDGE_AR_G:D3, H-BRIDGE_AR_G:D4, H-BRIDGE_AV_D:D1, H-BRIDGE_AV_D:D2, H-BRIDGE_AV_D:D3, H-BRIDGE_AV_D:D4, H-BRIDGE_AV_G:D1, H-BRIDGE_AV_G:D2, H-BRIDGE_AV_G:D3, H-BRIDGE_AV_G:D4: 1N4942, diode:DO41-10
- added H-BRIDGE_AR_D:IC1, H-BRIDGE_AR_G:IC1, H-BRIDGE_AV_D:IC1, H-BRIDGE_AV_G:IC1: L298, st-microelectronics:MULTIWATT-15
- added H-BRIDGE_AR_D:R1, H-BRIDGE_AR_D:R2, H-BRIDGE_AR_D:R3, H-BRIDGE_AR_G:R1, H-BRIDGE_AR_G:R2, H-BRIDGE_AR_G:R3, H-BRIDGE_AV_D:R1, H-BRIDGE_AV_D:R2, H-BRIDGE_AV_D:R3, H-BRIDGE_AV_G:R1, H-BRIDGE_AV_G:R2, H-BRIDGE_AV_G:R3, R8, R9: 10k, resistor:R0805
- added LED4: (no value), led:1206
- added R10: 330, resistor:R0805
- added RASPPBERRY_PI: (no value), pinhead:2X20/90
- added U$3: WIZ820IO, WIZnet:WIZ820
- added U1: TEENSY_3.5_DIL+USB, Teensy_libSG:TEENSY_3.5_DIL+USB
- added U2: TEENSY_3.1-3.2_DIL, Teensy_libSG:TEENSY_3.0-3.2&LC_DIL
- added XL320_D, XL320_G: DYNAMIXEL-1X03XL, 1NTech_pinhead:DYNAMIXEL_XL_1X03
- U$2: value TEENSY_3.5_DIL+USB -> PUSH-BUTTON; device Teensy_libSG:TEENSY_3.5_DIL+USB -> push-button:PUSH-BUTTON
- moved MOT_AR_D 864.3 mm to (46.0, 100.0), flipped to the bottom, turned to 180 degrees
- moved MOT_AR_G 860.5 mm to (83.0, 100.0), flipped to the bottom, turned to 180 degrees
- moved MOT_AV_D 831.2 mm to (46.0, 96.0), flipped to the bottom, turned to 180 degrees
- moved MOT_AV_G 827.8 mm to (83.0, 96.0), flipped to the bottom, turned to 180 degrees
- moved ENCODEUR_GAUCHE 802.4 mm to (79.0, 84.0), flipped to the bottom, turned to 180 degrees
- moved R5 798.2 mm to (125.0, 84.0), turned to 270 degrees
- moved ENCODEUR_DROIT 795.9 mm to (50.0, 84.0), flipped to the bottom, turned to 180 degrees
- moved LED3 786.8 mm to (127.0, 84.0), turned to 90 degrees
- moved R4 777.6 mm to (125.0, 68.0), turned to 90 degrees
- moved LED2 766.2 mm to (127.0, 68.0), turned to 90 degrees
- moved S3 759.7 mm to (126.0, 76.0), turned to 90 degrees
- moved R6 714.4 mm to (-38.0, 31.0)
- moved R7 713.7 mm to (-38.0, 24.0)
- moved Q2 713.7 mm to (-37.0, 38.0)
- moved S1 675.6 mm to (3.00, 93.0), turned to 270 degrees
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Connections:
- new net ENC_AR_D_A: MOT_AR_D.5
- new net ENC_AR_D_B: MOT_AR_D.6
- new net ENC_AR_G_A: MOT_AR_G.5
- new net ENC_AR_G_B: MOT_AR_G.6
- new net ENC_AV_D_A: MOT_AV_D.5
- new net ENC_AV_D_B: MOT_AV_D.6
- new net ENC_AV_G_A: MOT_AV_G.5
- new net ENC_AV_G_B: MOT_AV_G.6
- new net ETH_MISO: U$3.MISO
- new net ETH_MOSI: U$3.MOSI
- new net ETH_RST: R8.2, U$3.RESET
- new net ETH_SCLK: U$3.SCLK
- new net ETH_SS: U$3.SS
- new net N$10: GRUE.1
- new net N$11: LED4.A, R10.2
- new net N$5: R10.1, RASPPBERRY_PI.31
- new net N$6: GRUE.2
- new net N$9: LIPO.10, LIPO.11, LIPO.12, LIPO.7, LIPO.8, LIPO.9, P1.P$2
- net +12V: now also ARRET_URGENCE.10, ARRET_URGENCE.11, ARRET_URGENCE.12, ARRET_URGENCE.7, ARRET_URGENCE.8, ARRET_URGENCE.9, AX12_D.DYN_VCC, AX12_G.DYN_VCC, C5.+, C8.+, GRUE.10, GRUE.7, GRUE.8, GRUE.9, H-BRIDGE_AR_D:C1.2, H-BRIDGE_AR_D:D2.C, H-BRIDGE_AR_D:D4.C, H-BRIDGE_AR_D:IC1.4, H-BRIDGE_AR_G:C1.2, H-BRIDGE_AR_G:D2.C, H-BRIDGE_AR_G:D4.C, H-BRIDGE_AR_G:IC1.4, H-BRIDGE_AV_D:C1.2, H-BRIDGE_AV_D:D2.C, H-BRIDGE_AV_D:D4.C, H-BRIDGE_AV_D:IC1.4, H-BRIDGE_AV_G:C1.2, H-BRIDGE_AV_G:D2.C, H-BRIDGE_AV_G:D4.C, H-BRIDGE_AV_G:IC1.4; no longer ALIM-GRUE.1, H-BRIDGE1:C1.2, H-BRIDGE1:D2.C, H-BRIDGE1:D4.C, H-BRIDGE1:IC1.4, H-BRIDGE2:C1.2, H-BRIDGE2:D2.C, H-BRIDGE2:D4.C, H-BRIDGE2:IC1.4, H-BRIDGE3:C1.2, H-BRIDGE3:D2.C, H-BRIDGE3:D4.C, H-BRIDGE3:IC1.4, H-BRIDGE4:C1.2, H-BRIDGE4:D2.C, H-BRIDGE4:D4.C, H-BRIDGE4:IC1.4, LIPO-ET-ARRET-URGENCE.4
- net +3V3: now also R8.1, R9.1, U$3.VIN1, U$3.VIN2
- net +5V: now also H-BRIDGE_AR_D:C2.2, H-BRIDGE_AR_D:IC1.9, H-BRIDGE_AR_G:C2.2, H-BRIDGE_AR_G:IC1.9, H-BRIDGE_AV_D:C2.2, H-BRIDGE_AV_D:IC1.9, H-BRIDGE_AV_G:C2.2, H-BRIDGE_AV_G:IC1.9, MOT_AR_D.4, MOT_AR_G.4, MOT_AV_D.4, MOT_AV_G.4, RASPPBERRY_PI.2, RASPPBERRY_PI.4; no longer H-BRIDGE1:C2.2, H-BRIDGE1:IC1.9, H-BRIDGE2:C2.2, H-BRIDGE2:IC1.9, H-BRIDGE3:C2.2, H-BRIDGE3:IC1.9, H-BRIDGE4:C2.2, H-BRIDGE4:IC1.9
- net +6V5: now also C6.+, C7.+, XL320_D.VCC, XL320_G.VCC
- net 3.3V: now also U1.3.3V, U1.3.3V3, U2.3.3V; no longer U$1.3.3V, U$2.3.3V, U$2.3.3V3
- net AGND: now also U1.AGND, U2.AGND; no longer U$1.AGND, U$2.AGND
- net GND: now also AX12_D.GND, AX12_G.GND, C10.-, C5.-, C6.-, C7.-, C8.-, GRUE.3, GRUE.4, GRUE.5, GRUE.6, H-BRIDGE_AR_D:C1.1, H-BRIDGE_AR_D:C2.1, H-BRIDGE_AR_D:D1.A, H-BRIDGE_AR_D:D3.A, H-BRIDGE_AR_D:IC1.1, H-BRIDGE_AR_D:IC1.15, H-BRIDGE_AR_D:IC1.8, H-BRIDGE_AR_D:R1.2, H-BRIDGE_AR_D:R2.2, H-BRIDGE_AR_D:R3.2, H-BRIDGE_AR_G:C1.1, H-BRIDGE_AR_G:C2.1, H-BRIDGE_AR_G:D1.A, H-BRIDGE_AR_G:D3.A, H-BRIDGE_AR_G:IC1.1, H-BRIDGE_AR_G:IC1.15, H-BRIDGE_AR_G:IC1.8, H-BRIDGE_AR_G:R1.2, H-BRIDGE_AR_G:R2.2, H-BRIDGE_AR_G:R3.2, H-BRIDGE_AV_D:C1.1, H-BRIDGE_AV_D:C2.1, H-BRIDGE_AV_D:D1.A, H-BRIDGE_AV_D:D3.A, H-BRIDGE_AV_D:IC1.1, H-BRIDGE_AV_D:IC1.15, H-BRIDGE_AV_D:IC1.8, H-BRIDGE_AV_D:R1.2, H-BRIDGE_AV_D:R2.2, H-BRIDGE_AV_D:R3.2, H-BRIDGE_AV_G:C1.1, H-BRIDGE_AV_G:C2.1, H-BRIDGE_AV_G:D1.A, H-BRIDGE_AV_G:D3.A, H-BRIDGE_AV_G:IC1.1, H-BRIDGE_AV_G:IC1.15, H-BRIDGE_AV_G:IC1.8, H-BRIDGE_AV_G:R1.2, H-BRIDGE_AV_G:R2.2, H-BRIDGE_AV_G:R3.2, LED4.C, LIPO.1, LIPO.2, LIPO.3, LIPO.4, LIPO.5, LIPO.6, MOT_AR_D.3, MOT_AR_G.3, MOT_AV_D.3, MOT_AV_G.3, RASPPBERRY_PI.14, RASPPBERRY_PI.20, RASPPBERRY_PI.25, RASPPBERRY_PI.30, RASPPBERRY_PI.34, RASPPBERRY_PI.39, RASPPBERRY_PI.6, RASPPBERRY_PI.9, U$2.1, U$2.2, U$3.GND1, U$3.GND2, U$3.GND3, U$3.PWDN, U1.GND, U1.GND1, U2.GND, XL320_D.GND, XL320_G.GND; no longer ALIM-GRUE.2, H-BRIDGE1:C1.1, H-BRIDGE1:C2.1, H-BRIDGE1:D1.A, H-BRIDGE1:D3.A, H-BRIDGE1:IC1.1, H-BRIDGE1:IC1.15, H-BRIDGE1:IC1.8, H-BRIDGE1:R1.2, H-BRIDGE1:R2.2, H-BRIDGE1:R3.2, H-BRIDGE2:C1.1, H-BRIDGE2:C2.1, H-BRIDGE2:D1.A, H-BRIDGE2:D3.A, H-BRIDGE2:IC1.1, H-BRIDGE2:IC1.15, H-BRIDGE2:IC1.8, H-BRIDGE2:R1.2, H-BRIDGE2:R2.2, H-BRIDGE2:R3.2, H-BRIDGE3:C1.1, H-BRIDGE3:C2.1, H-BRIDGE3:D1.A, H-BRIDGE3:D3.A, H-BRIDGE3:IC1.1, H-BRIDGE3:IC1.15, H-BRIDGE3:IC1.8, H-BRIDGE3:R1.2, H-BRIDGE3:R2.2, H-BRIDGE3:R3.2, H-BRIDGE4:C1.1, H-BRIDGE4:C2.1, H-BRIDGE4:D1.A, H-BRIDGE4:D3.A, H-BRIDGE4:IC1.1, H-BRIDGE4:IC1.15, H-BRIDGE4:IC1.8, H-BRIDGE4:R1.2, H-BRIDGE4:R2.2, H-BRIDGE4:R3.2, LIPO-ET-ARRET-URGENCE.2, U$1.GND, U$2.GND, U$2.GND1
- net MOT_AR_D_EN: now also H-BRIDGE_AR_D:IC1.11, H-BRIDGE_AR_D:IC1.6, H-BRIDGE_AR_D:R1.1; no longer H-BRIDGE4:IC1.11, H-BRIDGE4:IC1.6, H-BRIDGE4:R1.1
- net MOT_AR_D_IN1: now also H-BRIDGE_AR_D:IC1.12, H-BRIDGE_AR_D:IC1.5, H-BRIDGE_AR_D:R2.1; no longer H-BRIDGE4:IC1.12, H-BRIDGE4:IC1.5, H-BRIDGE4:R2.1
- net MOT_AR_D_IN2: now also H-BRIDGE_AR_D:IC1.10, H-BRIDGE_AR_D:IC1.7, H-BRIDGE_AR_D:R3.1; no longer H-BRIDGE4:IC1.10, H-BRIDGE4:IC1.7, H-BRIDGE4:R3.1
- net MOT_AR_D_OUT+: now also H-BRIDGE_AR_D:D1.C, H-BRIDGE_AR_D:D2.A, H-BRIDGE_AR_D:IC1.14, H-BRIDGE_AR_D:IC1.2, MOT_AR_D.1; no longer H-BRIDGE4:D1.C, H-BRIDGE4:D2.A, H-BRIDGE4:IC1.14, H-BRIDGE4:IC1.2
- net MOT_AR_D_OUT-: now also H-BRIDGE_AR_D:D3.C, H-BRIDGE_AR_D:D4.A, H-BRIDGE_AR_D:IC1.13, H-BRIDGE_AR_D:IC1.3, MOT_AR_D.2; no longer H-BRIDGE4:D3.C, H-BRIDGE4:D4.A, H-BRIDGE4:IC1.13, H-BRIDGE4:IC1.3
- net MOT_AR_G_EN: now also H-BRIDGE_AR_G:IC1.11, H-BRIDGE_AR_G:IC1.6, H-BRIDGE_AR_G:R1.1; no longer H-BRIDGE3:IC1.11, H-BRIDGE3:IC1.6, H-BRIDGE3:R1.1
- net MOT_AR_G_IN1: now also H-BRIDGE_AR_G:IC1.12, H-BRIDGE_AR_G:IC1.5, H-BRIDGE_AR_G:R2.1; no longer H-BRIDGE3:IC1.12, H-BRIDGE3:IC1.5, H-BRIDGE3:R2.1
- net MOT_AR_G_IN2: now also H-BRIDGE_AR_G:IC1.10, H-BRIDGE_AR_G:IC1.7, H-BRIDGE_AR_G:R3.1; no longer H-BRIDGE3:IC1.10, H-BRIDGE3:IC1.7, H-BRIDGE3:R3.1
- net MOT_AR_G_OUT+: now also H-BRIDGE_AR_G:D1.C, H-BRIDGE_AR_G:D2.A, H-BRIDGE_AR_G:IC1.14, H-BRIDGE_AR_G:IC1.2, MOT_AR_G.1; no longer H-BRIDGE3:D1.C, H-BRIDGE3:D2.A, H-BRIDGE3:IC1.14, H-BRIDGE3:IC1.2
- net MOT_AR_G_OUT-: now also H-BRIDGE_AR_G:D3.C, H-BRIDGE_AR_G:D4.A, H-BRIDGE_AR_G:IC1.13, H-BRIDGE_AR_G:IC1.3, MOT_AR_G.2; no longer H-BRIDGE3:D3.C, H-BRIDGE3:D4.A, H-BRIDGE3:IC1.13, H-BRIDGE3:IC1.3
- net MOT_AV_D_EN: now also H-BRIDGE_AV_D:IC1.11, H-BRIDGE_AV_D:IC1.6, H-BRIDGE_AV_D:R1.1; no longer H-BRIDGE2:IC1.11, H-BRIDGE2:IC1.6, H-BRIDGE2:R1.1
- net MOT_AV_D_IN1: now also H-BRIDGE_AV_D:IC1.12, H-BRIDGE_AV_D:IC1.5, H-BRIDGE_AV_D:R2.1; no longer H-BRIDGE2:IC1.12, H-BRIDGE2:IC1.5, H-BRIDGE2:R2.1
- net MOT_AV_D_IN2: now also H-BRIDGE_AV_D:IC1.10, H-BRIDGE_AV_D:IC1.7, H-BRIDGE_AV_D:R3.1; no longer H-BRIDGE2:IC1.10, H-BRIDGE2:IC1.7, H-BRIDGE2:R3.1
- net MOT_AV_D_OUT+: now also H-BRIDGE_AV_D:D1.C, H-BRIDGE_AV_D:D2.A, H-BRIDGE_AV_D:IC1.14, H-BRIDGE_AV_D:IC1.2, MOT_AV_D.1; no longer H-BRIDGE2:D1.C, H-BRIDGE2:D2.A, H-BRIDGE2:IC1.14, H-BRIDGE2:IC1.2
- net MOT_AV_D_OUT-: now also H-BRIDGE_AV_D:D3.C, H-BRIDGE_AV_D:D4.A, H-BRIDGE_AV_D:IC1.13, H-BRIDGE_AV_D:IC1.3, MOT_AV_D.2; no longer H-BRIDGE2:D3.C, H-BRIDGE2:D4.A, H-BRIDGE2:IC1.13, H-BRIDGE2:IC1.3
- net MOT_AV_G_EN: now also H-BRIDGE_AV_G:IC1.11, H-BRIDGE_AV_G:IC1.6, H-BRIDGE_AV_G:R1.1; no longer H-BRIDGE1:IC1.11, H-BRIDGE1:IC1.6, H-BRIDGE1:R1.1
- net MOT_AV_G_IN1: now also H-BRIDGE_AV_G:IC1.12, H-BRIDGE_AV_G:IC1.5, H-BRIDGE_AV_G:R2.1; no longer H-BRIDGE1:IC1.12, H-BRIDGE1:IC1.5, H-BRIDGE1:R2.1
- net MOT_AV_G_IN2: now also H-BRIDGE_AV_G:IC1.10, H-BRIDGE_AV_G:IC1.7, H-BRIDGE_AV_G:R3.1; no longer H-BRIDGE1:IC1.10, H-BRIDGE1:IC1.7, H-BRIDGE1:R3.1
- net MOT_AV_G_OUT+: now also H-BRIDGE_AV_G:D1.C, H-BRIDGE_AV_G:D2.A, H-BRIDGE_AV_G:IC1.14, H-BRIDGE_AV_G:IC1.2, MOT_AV_G.1; no longer H-BRIDGE1:D1.C, H-BRIDGE1:D2.A, H-BRIDGE1:IC1.14, H-BRIDGE1:IC1.2
- net MOT_AV_G_OUT-: now also H-BRIDGE_AV_G:D3.C, H-BRIDGE_AV_G:D4.A, H-BRIDGE_AV_G:IC1.13, H-BRIDGE_AV_G:IC1.3, MOT_AV_G.2; no longer H-BRIDGE1:D3.C, H-BRIDGE1:D4.A, H-BRIDGE1:IC1.13, H-BRIDGE1:IC1.3
- net N$2: now also R9.2, RASPPBERRY_PI.29, U$2.3, U$2.4; no longer LIPO-ET-ARRET-URGENCE.1, P1.P$2
- net N$3: now also ARRET_URGENCE.1, ARRET_URGENCE.2, ARRET_URGENCE.3, ARRET_URGENCE.4, ARRET_URGENCE.5, ARRET_URGENCE.6, C10.+; no longer LIPO-ET-ARRET-URGENCE.3
- net SERIAL_AX12_5V: now also AX12_D.DATA, AX12_G.DATA
- net SERIAL_XL320_5V: now also XL320_D.DATA, XL320_G.DATA
- net VIN: now also U1.VIN, U2.VIN; no longer U$1.VIN, U$2.VIN
Other:
- board size 160 x 100 mm -> 129 x 106 mm

Commit message: pin mapping teensy
Parts:
- added JUMPER: JST-03, con-jst:GH-03-V
- added LED5, LED6: (no value), led:1206
- added R11: 22k, resistor:R0805
- added R12: 6k8, resistor:R0805
- added R13, R14: 330, resistor:R0805
Connections:
- removed net 3.3V: U1.3.3V, U1.3.3V3, U2.3.3V
- removed net AGND: U1.AGND, U2.AGND
- new net DEL_CLIGNOTANT_D: DELS_ET_TOF_AR.11, PHARES_ET_TOF_AV.9
- new net DEL_CLIGNOTANT_G: DELS_ET_TOF_AR.12, PHARES_ET_TOF_AV.8
- new net DEL_FEUX_NUIT_AR: DELS_ET_TOF_AR.13
- new net DEL_FEUX_NUIT_AV: PHARES_ET_TOF_AV.10
- new net DEL_FEUX_RECUL: DELS_ET_TOF_AR.15
- new net DEL_FEUX_STOP: DELS_ET_TOF_AR.14
- new net DEL_GYRO_1: DEL_GYRO.2
- new net DEL_GYRO_2: DEL_GYRO.3
- new net DEL_GYRO_3: DEL_GYRO.4
- new net DEL_GYRO_4: DEL_GYRO.5
- new net ENC_D_A: ENCODEUR_DROIT.3, U1.18/A4
- new net ENC_D_B: ENCODEUR_DROIT.4, U1.39/A20
- new net ENC_G_A: ENCODEUR_GAUCHE.3, U1.16/A2
- new net ENC_G_B: ENCODEUR_GAUCHE.4, U1.17/A3
- new net GRUE_SERIAL_MISO: GRUE.2, U1.0
- new net GRUE_SERIAL_MOSI: GRUE.1, U1.1
- new net JUMPER: JUMPER.3, U1.19/A5
- new net N$12: R11.2, R12.1, U1.A21
- new net N$13: LED6.A, R14.1
- new net N$14: LED5.A, R13.1
- new net N$15: R13.2, U1.14/A0
- new net N$16: R14.2, U1.20/A6
- new net N$19: U2.8
- new net N$20: U2.11
- new net N$21: U2.12
- new net N$22: U2.14/A0
- new net N$23: U2.15/A1
- new net N$24: U2.16/A2
- new net N$25: U2.17/A3
- new net SCL: DELS_ET_TOF_AR.4, PHARES_ET_TOF_AV.4, U2.19/A5
- new net SDA: DELS_ET_TOF_AR.3, PHARES_ET_TOF_AV.3, U2.18/A4
- new net TOF_AR_D: DELS_ET_TOF_AR.7
- new net TOF_AR_G: DELS_ET_TOF_AR.8
- new net TOF_AV: PHARES_ET_TOF_AV.6
- new net TOF_AV_D: PHARES_ET_TOF_AV.7, U2.7
- new net TOF_AV_G: PHARES_ET_TOF_AV.5, U2.2
- new net TOF_FLAN_AR_D: DELS_ET_TOF_AR.6
- new net TOF_FLAN_AR_G: DELS_ET_TOF_AR.9
- new net TOF_FLAN_AV_D: DELS_ET_TOF_AR.5
- new net TOF_FLAN_AV_G: DELS_ET_TOF_AR.10
- net +12V: now also R11.1
- net +3V3: now also DELS_ET_TOF_AR.2, JUMPER.2, PHARES_ET_TOF_AV.2, U1.3.3V, U1.3.3V3, U2.3.3V
- net +5V: now also ENCODEUR_DROIT.1, ENCODEUR_GAUCHE.1
- net CHOOSE_COLOR: now also U1.A22
- net ENC_AR_D_A: now also U1.30
- net ENC_AR_D_B: now also U1.38/A19
- net ENC_AR_G_A: now also U1.28
- net ENC_AR_G_B: now also U1.29
- net ENC_AV_D_A: now also U1.26
- net ENC_AV_D_B: now also U1.27
- net ENC_AV_G_A: now also U1.24
- net ENC_AV_G_B: now also U1.25
- net ETH_MISO: now also U1.12
- net ETH_MOSI: now also U1.11
- net ETH_RST: now also U1.15/A1
- net ETH_SCLK: now also U1.13
- net ETH_SS: now also U1.10
- net GND: now also DELS_ET_TOF_AR.1, DEL_GYRO.1, ENCODEUR_DROIT.2, ENCODEUR_GAUCHE.2, JUMPER.1, LED5.C, LED6.C, PHARES_ET_TOF_AV.1, R12.2, U1.AGND, U2.AGND
- net MOT_AR_D_EN: now also U1.35/A16
- net MOT_AR_D_IN1: now also U1.36/A17
- net MOT_AR_D_IN2: now also U1.37/A18
- net MOT_AR_G_EN: now also U1.21/A7
- net MOT_AR_G_IN1: now also U1.22/A8
- net MOT_AR_G_IN2: now also U1.23/A9
- net MOT_AV_D_EN: now also U1.5
- net MOT_AV_D_IN1: now also U1.6
- net MOT_AV_D_IN2: now also U1.9
- net MOT_AV_G_EN: now also U1.2
- net MOT_AV_G_IN1: now also U1.3
- net MOT_AV_G_IN2: now also U1.4
- net N$10: now also U1.34/A15, U2.1; no longer GRUE.1
- net N$6: now also U1.33/A14, U2.0; no longer GRUE.2
- net SERIAL_AX12: now also U1.7, U1.8
- net SERIAL_XL320: now also U1.31/A12, U1.32/A13

Commit message: Début de routage...
Parts:
- added R15, R17, R20, R22, R24, R26, R28, R30, R32, R34: 0, resistor:R0805
- added R16, R18, R19, R21, R23, R25, R27, R29, R31, R33: 270, resistor:R0805
- added T1, T10, T2, T3, T4, T5, T6, T7, T8, T9: (no value), transistor:SOT23-BEC
- C1, C2, C3, C4: value (none) -> 10µF
- C10: value (none) -> 4700µF
- H-BRIDGE_AR_D:C1, H-BRIDGE_AR_D:C2, H-BRIDGE_AR_G:C1, H-BRIDGE_AR_G:C2, H-BRIDGE_AV_D:C1, H-BRIDGE_AV_D:C2, H-BRIDGE_AV_G:C1, H-BRIDGE_AV_G:C2: value (none) -> 100nF
- H-BRIDGE_AR_D:D1, H-BRIDGE_AR_D:D2, H-BRIDGE_AR_D:D3, H-BRIDGE_AR_D:D4, H-BRIDGE_AR_G:D1, H-BRIDGE_AR_G:D2, H-BRIDGE_AR_G:D3, H-BRIDGE_AR_G:D4, H-BRIDGE_AV_D:D1, H-BRIDGE_AV_D:D2, H-BRIDGE_AV_D:D3, H-BRIDGE_AV_D:D4, H-BRIDGE_AV_G:D1, H-BRIDGE_AV_G:D2, H-BRIDGE_AV_G:D3, H-BRIDGE_AV_G:D4: value 1N4942 -> S1M; device diode:DO41-10 -> diode:SMA
- LED1, LED5: value (none) -> blue
- LED2: value (none) -> green
- LED3: value (none) -> orange
- LED4, LED6: value (none) -> red
- moved JUMPER 173.7 mm to (64.5, 100.0), flipped to the bottom, turned to 180 degrees
- moved DC2 159.0 mm to (123.0, 89.0)
- moved DC4 158.5 mm to (112.0, 98.0)
- moved H-BRIDGE_AR_G:D2 157.0 mm to (112.0, 75.0), turned to 270 degrees
- moved H-BRIDGE_AR_G:D1 154.0 mm to (109.0, 75.0), turned to 90 degrees
- moved H-BRIDGE_AR_G:D3 150.1 mm to (105.0, 75.0), turned to 270 degrees
- moved H-BRIDGE_AR_G:D4 147.2 mm to (102.0, 75.0), turned to 90 degrees
- moved DC1 145.1 mm to (121.0, 55.0), turned to 270 degrees
- moved C4 141.8 mm to (102.0, 100.0), turned to 90 degrees
- moved C2 140.9 mm to (113.0, 91.0), turned to 90 degrees
- moved LED6 140.5 mm to (2.00, 61.0), turned to 270 degrees
- moved R14 137.6 mm to (5.00, 63.0)
- moved LED5 135.2 mm to (2.00, 69.0), turned to 270 degrees
- moved R13 132.4 mm to (5.00, 71.0)
- moved R12 130.7 mm to (43.0, 40.0), turned to 270 degrees
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Connections:
- removed net N$19: U2.8
- removed net N$20: U2.11
- removed net N$23: U2.15/A1
- removed net N$24: U2.16/A2
- new net DEL_CLIGNOTANT_D_PWM: R27.1, U2.20/A6
- new net DEL_CLIGNOTANT_G_PWM: R25.1, U2.10
- new net DEL_FEUX_NUIT_AR_PWM: R29.1, U2.21/A7
- new net DEL_FEUX_NUIT_AV_PWM: R23.1, U2.9
- new net DEL_FEUX_RECUL_PWM: R33.1, U2.23/A9
- new net DEL_FEUX_STOP_PWM: R31.1, U2.22/A8
- new net DEL_GYRO_1_PWM: R19.1, U2.3
- new net DEL_GYRO_2_PWM: R16.1, U2.4
- new net DEL_GYRO_3_PWM: R18.1, U2.5
- new net DEL_GYRO_4_PWM: R21.1, U2.6
- new net N$17: R15.1, T3.E
- new net N$18: R19.2, T3.B
- new net N$26: R18.2, T2.B
- new net N$29: R22.1, T4.E
- new net N$30: R21.2, T4.B
- new net N$33: R24.1, T5.E
- new net N$34: R23.2, T5.B
- new net N$37: R26.1, T6.E
- new net N$38: R25.2, T6.B
- new net N$41: R28.1, T7.E
- new net N$42: R27.2, T7.B
- new net N$45: R30.1, T8.E
- new net N$46: R29.2, T8.B
- new net N$49: R32.1, T9.E
- new net N$50: R31.2, T9.B
- new net N$53: R34.1, T10.E
- new net N$54: R33.2, T10.B
- net +12V: now also H-BRIDGE_AR_D:D3.C, H-BRIDGE_AR_G:D3.C, H-BRIDGE_AV_D:D3.C, H-BRIDGE_AV_G:D3.C; no longer H-BRIDGE_AR_D:D4.C, H-BRIDGE_AR_G:D4.C, H-BRIDGE_AV_D:D4.C, H-BRIDGE_AV_G:D4.C
- net +3V3_LEDS: now also T1.C, T10.C, T2.C, T3.C, T4.C, T5.C, T6.C, T7.C, T8.C, T9.C
- net DEL_CLIGNOTANT_D: now also R28.2
- net DEL_CLIGNOTANT_G: now also R26.2
- net DEL_FEUX_NUIT_AR: now also R30.2
- net DEL_FEUX_NUIT_AV: now also R24.2
- net DEL_FEUX_RECUL: now also R34.2
- net DEL_FEUX_STOP: now also R32.2
- net DEL_GYRO_1: now also R15.2
- net DEL_GYRO_2: now also R17.2
- net DEL_GYRO_3: now also R20.2
- net DEL_GYRO_4: now also R22.2
- net GND: now also H-BRIDGE_AR_D:D4.A, H-BRIDGE_AR_G:D4.A, H-BRIDGE_AV_D:D4.A, H-BRIDGE_AV_G:D4.A, S1.B, S1.B1; no longer H-BRIDGE_AR_D:D3.A, H-BRIDGE_AR_G:D3.A, H-BRIDGE_AV_D:D3.A, H-BRIDGE_AV_G:D3.A
- net MOT_AR_D_OUT-: now also H-BRIDGE_AR_D:D3.A, H-BRIDGE_AR_D:D4.C; no longer H-BRIDGE_AR_D:D3.C, H-BRIDGE_AR_D:D4.A
- net MOT_AR_G_OUT-: now also H-BRIDGE_AR_G:D3.A, H-BRIDGE_AR_G:D4.C; no longer H-BRIDGE_AR_G:D3.C, H-BRIDGE_AR_G:D4.A
- net MOT_AV_D_OUT-: now also H-BRIDGE_AV_D:D3.A, H-BRIDGE_AV_D:D4.C; no longer H-BRIDGE_AV_D:D3.C, H-BRIDGE_AV_D:D4.A
- net MOT_AV_G_OUT-: now also H-BRIDGE_AV_G:D3.A, H-BRIDGE_AV_G:D4.C; no longer H-BRIDGE_AV_G:D3.C, H-BRIDGE_AV_G:D4.A
- net N$21: now also R17.1, T1.E; no longer U2.12
- net N$22: now also R16.2, T1.B; no longer U2.14/A0
- net N$25: now also R20.1, T2.E; no longer U2.17/A3
- net TOF_AR_D: now also U2.14/A0
- net TOF_AR_G: now also U2.15/A1
- net TOF_AV: now also U2.7
- net TOF_AV_D: now also U2.8; no longer U2.7
- net TOF_FLAN_AR_D: now also U2.12
- net TOF_FLAN_AR_G: now also U2.16/A2
- net TOF_FLAN_AV_D: now also U2.11
- net TOF_FLAN_AV_G: now also U2.17/A3
Routing:
- net +12V: track 0.00 -> 347.5 mm, vias 0 -> 18
- net GND: track 0.00 -> 138.0 mm
- net MOT_AR_G_OUT+: track 0.00 -> 134.1 mm
- net MOT_AR_G_OUT-: track 0.00 -> 118.5 mm
- net MOT_AR_D_OUT+: track 0.00 -> 117.5 mm, vias 0 -> 1
- net MOT_AR_D_OUT-: track 0.00 -> 109.6 mm, vias 0 -> 1
- net N$3: track 0.00 -> 94.1 mm, vias 0 -> 3
- net MOT_AV_G_OUT+: track 0.00 -> 84.4 mm
- net MOT_AV_G_OUT-: track 0.00 -> 74.2 mm, vias 0 -> 1
- net MOT_AV_D_OUT+: track 0.00 -> 73.6 mm
- net MOT_AV_D_OUT-: track 0.00 -> 67.9 mm, vias 0 -> 1
- net +5V: track 0.00 -> 33.1 mm
- net MOT_AV_D_EN: track 0.00 -> 25.8 mm, vias 0 -> 1
- net CHOOSE_COLOR: track 0.00 -> 22.7 mm
- net MOT_AV_D_IN1: track 0.00 -> 22.1 mm, vias 0 -> 1
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
Commit message: ajout carte elec grue
Parts:
- C1, C2, C3, C4: device resistor:E2,5-7 -> resistor:C0805
- C5, C6, C7, C8: device resistor:E2,5-6 -> resistor:C0805
- moved C4 10.0 mm to (110.0, 94.0), turned to 0 degrees
- moved C1 3.00 mm to (118.0, 56.0)
- moved C3 2.83 mm to (30.0, 103.0)
- moved DC3 2.00 mm to (20.0, 102.0)
- moved DC4 1.00 mm to (111.0, 98.0)
- moved C8 0.90 mm to (93.1, 85.0)
- moved C5 0.90 mm to (35.9, 83.0)
Connections:
- net +12V: now also C1.1, C2.1, C4.1, C5.1, C8.1; no longer C1.+, C2.+, C4.+, C5.+, C8.+
- net +6V5: now also C6.1, C7.1; no longer C6.+, C7.+
- net 12V_AUX: now also C3.1; no longer C3.+
- net GND: now also C1.2, C2.2, C3.2, C4.2, C5.2, C6.2, C7.2, C8.2; no longer C1.-, C2.-, C3.-, C4.-, C5.-, C6.-, C7.-, C8.-
Routing:
- net +12V: track 347.5 -> 340.6 mm, vias 18 -> 19
- net +5V: track 33.1 -> 35.1 mm
- net 12V_AUX: track 15.7 -> 16.7 mm
