File: electronique/camion-grue.brd (EAGLE design)
At the start: 129 x 106 mm, 132 parts, among them P1 RGEF800, Q1 BSS138, Q2 BSS138, U1 TEENSY_3.5_DIL+USB, U2 TEENSY_3.1-3.2_DIL

Commit message: Elec robot: régulateur 5V dédié pour la logique, indépendant de celui de la RPI
Parts:
- added C11: 22µF, resistor:C0805
- added C9: 10µF, resistor:C0805
- added IC3: REG1117, burr-brown:SOT223
Connections:
- new net +5V_RPI: DC3.3, R1.2, RASPPBERRY_PI.2, RASPPBERRY_PI.4
- net +12V: now also C9.1, IC3.3
- net +5V: now also C11.1, IC3.2; no longer DC3.3, R1.2, RASPPBERRY_PI.2, RASPPBERRY_PI.4
- net GND: now also C11.2, C9.2, IC3.1
Routing:
- net +5V_RPI: track 0.00 -> 125.7 mm
- net +5V: track 369.3 -> 278.7 mm, vias 9 -> 7
- net +12V: track 348.1 -> 370.8 mm, vias 19 -> 20
- net GND: vias 78 -> 81
