File: electronique/camion-grue.sch (EAGLE design)
At the start: 12 parts

Commit message: Ajout libs Eagle
Parts:
- added ALIM-GRUE: JST-02VL-V, con-jst:JST-02VL-V
- added D1: DIODE_S15P45, diode_schottky:DIODE_S15P45
- added LIPO-ET-ARRET-URGENCE: JST-04VL-V, con-jst:JST-04VL-V
- added P1: RGEF800, polyswitch:RGEF800
- added S1: (no value), switch:SWITCH_LPV-1
Connections:
- new net N$2: LIPO-ET-ARRET-URGENCE.1, P1.2
- new net N$3: D1.-, LIPO-ET-ARRET-URGENCE.3, S1.P
- new net N$4: D1.+, P1.1
- new net OUT+: D1.C
- net +12V: now also ALIM-GRUE.1, LIPO-ET-ARRET-URGENCE.4
- net 12V_AUX: now also S1.S
- net GND: now also ALIM-GRUE.2, D1.A, LIPO-ET-ARRET-URGENCE.2
Changed lines of the file:
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@@
 <part name="R1" library="resistor" library_urn="urn:adsk.eagle:library:348" deviceset="R-EU_" device="R0805" package3d_urn="urn:adsk.eagle:package:26059/1"/>
 <part name="SUPPLY21" library="supply2" library_urn="urn:adsk.eagle:library:372" deviceset="GND" device=""/>
+<part name="D1" library="diode_schottky" deviceset="DIODE_S15P45" device=""/>
+<part name="SUPPLY22" library="supply2" library_urn="urn:adsk.eagle:library:372" deviceset="GND" device=""/>
+<part name="SUPPLY23" library="supply2" library_urn="urn:adsk.eagle:library:372" deviceset="+12V" device=""/>
+<part name="P1" library="polyswitch" deviceset="RGEF800" device=""/>
+<part name="ALIM-GRUE" library="con-jst" deviceset="JST-02" device="VL-V"/>
+<part name="SUPPLY24" library="supply2" library_urn="urn:adsk.eagle:library:372" deviceset="+12V" device=""/>
+<part name="SUPPLY25" library="supply2" library_urn="urn:adsk.eagle:library:372" deviceset="GND" device=""/>
+<part name="LIPO-ET-ARRET-URGENCE" library="con-jst" deviceset="JST-04" device="VL-V"/>
+<part name="S1" library="switch" deviceset="SWITCH_LPV-1" device="">
+<attribute name="RS" value="734-7306"/>
+</part>
 </parts>
 <sheets>
@@
 <instance part="R1" gate="G$1" x="129.54" y="185.42" rot="R180"/>
 <instance part="SUPPLY21" gate="GND" x="149.86" y="185.42" rot="R90"/>
+<instance part="D1" gate="G$1" x="91.44" y="132.08" rot="R90"/>
+<instance part="SUPPLY22" gate="GND" x="101.6" y="132.08"/>
+<instance part="SUPPLY23" gate="+12V" x="109.22" y="124.46" rot="R180"/>
+<instance part="P1" gate="G$1" x="96.52" y="139.7"/>
+<instance part="ALIM-GRUE" gate="G$1" x="116.84" y="96.52"/>
+<instance part="SUPPLY24" gate="+12V" x="106.68" y="96.52" rot="R90"/>
+<instance part="SUPPLY25" gate="GND" x="106.68" y="93.98" rot="R270"/>
+<instance part="LIPO-ET-ARRET-URGENCE" gate="G$1" x="116.84" y="139.7"/>
+<instance part="S1" gate="1" x="101.6" y="111.76" rot="R270">
+<attribute name="RS" x="101.6" y="111.76" size="1.27" layer="96" rot="R270" display="off"/>
+</instance>
 </instances>
 <busses>
@@
 <pinref part="SUPPLY20" gate="+12V" pin="+12V"/>
 </segment>
+<segment>
+<pinref part="ALIM-GRUE" gate="G$1" pin="1"/>
+<wire x1="111.76" y1="96.52" x2="109.22" y2="96.52" width="0.1524" layer="91"/>
+<pinref part="SUPPLY24" gate="+12V" pin="+12V"/>
+</segment>
+<segment>
+<pinref part="LIPO-ET-ARRET-URGENCE" gate="G$1" pin="4"/>
+<wire x1="111.76" y1="132.08" x2="109.22" y2="132.08" width="0.1524" layer="91"/>
+<wire x1="109.22" y1="132.08" x2="109.22" y2="127" width="0.1524" layer="91"/>
+<pinref part="SUPPLY23" gate="+12V" pin="+12V"/>
+</segment>
 </net>
 <net name="GND" class="0">
@@
 <pinref part="SUPPLY21" gate="GND" pin="GND"/>
 <wire x1="147.32" y1="185.42" x2="144.78" y2="185.42" width="0.1524" layer="91"/>
+</segment>
+<segment>
+<pinref part="SUPPLY22" gate="GND" pin="GND"/>
+<wire x1="101.6" y1="134.62" x2="101.6" y2="137.16" width="0.1524" layer="91"/>
+<wire x1="101.6" y1="137.16" x2="111.76" y2="137.16" width="0.1524" layer="91"/>
+<pinref part="LIPO-ET-ARRET-URGENCE" gate="G$1" pin="2"/>
+</segment>
+<segment>
+<pinref part="ALIM-GRUE" gate="G$1" pin="2"/>
+<wire x1="111.76" y1="93.98" x2="109.22" y2="93.98" width="0.1524" layer="91"/>
+<pinref part="SUPPLY25" gate="GND" pin="GND"/>
 </segment>
 </net>
@@
 <label x="91.44" y="190.5" size="1.27" layer="95" rot="R180" xref="yes"/>
 </segment>
+<segment>
+<pinref part="S1" gate="1" pin="S"/>
+<wire x1="106.68" y1="106.68" x2="111.76" y2="106.68" width="0.1524" layer="91"/>
+<label x="111.76" y="106.68" size="1.27" layer="95" xref="yes"/>
+</segment>
 </net>
 <net name="+6V5" class="0">
@@
 </segment>
 </net>
+<net name="N$3" class="0">
+<segment>
+<wire x1="91.44" y1="127" x2="104.14" y2="127" width="0.1524" layer="91"/>
+<wire x1="91.44" y1="127" x2="91.44" y2="109.22" width="0.1524" layer="91"/>
+<wire x1="91.44" y1="109.22" x2="96.52" y2="109.22" width="0.1524" layer="91"/>
+<pinref part="D1" gate="G$1" pin="-"/>
+<wire x1="91.44" y1="129.54" x2="91.44" y2="127" width="0.1524" layer="91"/>
+<junction x="91.44" y="127"/>
+<wire x1="104.14" y1="127" x2="106.68" y2="127" width="0.1524" layer="91"/>
+<wire x1="106.68" y1="127" x2="106.68" y2="134.62" width="0.1524" layer="91"/>
+<pinref part="LIPO-ET-ARRET-URGENCE" gate="G$1" pin="3"/>
+<wire x1="106.68" y1="134.62" x2="111.76" y2="134.62" width="0.1524" layer="91"/>
+<pinref part="S1" gate="1" pin="P"/>
+</segment>
+</net>
+<net name="N$2" class="0">
+<segment>
+<pinref part="P1" gate="G$1" pin="2"/>
+<wire x1="101.6" y1="139.7" x2="111.76" y2="139.7" width="0.1524" layer="91"/>
+<pinref part="LIPO-ET-ARRET-URGENCE" gate="G$1" pin="1"/>
+</segment>
+</net>
+<net name="N$4" class="0">
+<segment>
+<pinref part="P1" gate="G$1" pin="1"/>
+<pinref part="D1" gate="G$1" pin="+"/>
+<wire x1="91.44" y1="139.7" x2="91.44" y2="137.16" width="0.1524" layer="91"/>
+</segment>
+</net>

Commit message: maj elec et libs eagle
Parts:
- added ENCODEUR_DROIT, ENCODEUR_GAUCHE: JST-04GH-V, con-jst:JST-04GH-V
- added FEUX_ARRIERE: JST-06, con-jst:JST-06
- added LED2, LED3: (no value), led:LEDSMT1206
- added MOT_AR_D, MOT_AR_G, MOT_AV_D, MOT_AV_G: (no value), pinhead:PINHD-1X6
- added Q1, Q2: BSS138, transistor-small-signal:BSS123
- added R2, R3, R6, R7: 10k, resistor:R-EU_R0805
- added R4, R5: 330, resistor:R-EU_R0805
- added S3: TL36PO, switch:TL36PO
- added SERIAL_GRUE: JST-02GH-V, con-jst:JST-02GH-V
- added TOF_FLAN_AV_D, TOF_FLAN_AV_G: JST-05, con-jst:JST-05
- R1: value (none) -> 470
Connections:
- new net CHOOSE_COLOR: LED3.C, R4.2, S3.P
- new net INPUT1: R2.1
- new net INPUT2: R3.1
- new net N$7: LED2.A, R4.1
- new net N$8: LED3.A, R5.2
- new net SERIAL_AX12: Q1.S, R2.2
- new net SERIAL_AX12_5V: Q1.D, R3.2
- new net SERIAL_XL320: Q2.S, R6.2
- new net SERIAL_XL320_5V: Q2.D, R7.2
- net +3V3: now also Q1.G, Q2.G, R2.1, R5.1, R6.1, S3.S
- net +5V: now also R3.1, R7.1
- net GND: now also LED2.C, R2.2, R3.2, S3.O

Commit message: Elec: schéma presque ok + placement des composants
Parts:
- removed ALIM-GRUE: JST-02VL-V, con-jst:JST-02VL-V
- removed FEUX_ARRIERE: JST-06, con-jst:JST-06
- removed LIPO-ET-ARRET-URGENCE: JST-04VL-V, con-jst:JST-04VL-V
- removed SERIAL_GRUE: JST-02GH-V, con-jst:JST-02GH-V
- removed TOF_FLAN_AV_D, TOF_FLAN_AV_G: JST-05, con-jst:JST-05
- removed U$1: TEENSY_3.1-3.2_DIL, Teensy_libSG:TEENSY_3.1-3.2_DIL
- added ARRET_URGENCE, LIPO: JST-12, con-jst:JST-12
- added AX12_D, AX12_G: DYNAMIXEL-1X03AX, 1NTech_pinhead:DYNAMIXEL-1X03AX
- added C10: (no value), 1NTech_RLCD:CPOL-EUTT5D11L
- added C5, C6, C7, C8: 1µF, resistor:CPOL-EUE2.5-6
- added DELS_ET_TOF_AR: JST-15, con-jst:JST-15
- added DEL_GYRO: JST-05, con-jst:JST-05
- added GRUE, PHARES_ET_TOF_AV: JST-10, con-jst:JST-10
- added LED4: (no value), led:LEDSMT1206
- added R10: 330, resistor:R-EU_R0805
- added R8, R9: 10k, resistor:R-EU_R0805
- added RASPPBERRY_PI: (no value), pinhead:PINHD-2X20/90
- added U$3: WIZ820IO, WIZnet:WIZ820IO
- added U1: TEENSY_3.5_DIL+USB, Teensy_libSG:TEENSY_3.5_DIL+USB
- added U2: TEENSY_3.1-3.2_DIL, Teensy_libSG:TEENSY_3.1-3.2_DIL
- added XL320_D, XL320_G: DYNAMIXEL-1X03XL, 1NTech_pinhead:DYNAMIXEL-1X03XL
- U$2: value TEENSY_3.5_DIL+USB -> PUSH-BUTTON; device Teensy_libSG:TEENSY_3.5_DIL+USB -> push-button:PUSH-BUTTON
Connections:
- new net ENC_AR_D_A: MOT_AR_D.5
- new net ENC_AR_D_B: MOT_AR_D.6
- new net ENC_AR_G_A: MOT_AR_G.5
- new net ENC_AR_G_B: MOT_AR_G.6
- new net ENC_AV_D_A: MOT_AV_D.5
- new net ENC_AV_D_B: MOT_AV_D.6
- new net ENC_AV_G_A: MOT_AV_G.5
- new net ENC_AV_G_B: MOT_AV_G.6
- new net ETH_MISO: U$3.MISO
- new net ETH_MOSI: U$3.MOSI
- new net ETH_RST: R8.2, U$3.RESET
- new net ETH_SCLK: U$3.SCLK
- new net ETH_SS: U$3.SS
- new net MOT_AR_D_OUT+: MOT_AR_D.1
- new net MOT_AR_D_OUT-: MOT_AR_D.2
- new net MOT_AR_G_OUT+: MOT_AR_G.1
- new net MOT_AR_G_OUT-: MOT_AR_G.2
- new net MOT_AV_D_OUT+: MOT_AV_D.1
- new net MOT_AV_D_OUT-: MOT_AV_D.2
- new net MOT_AV_G_OUT+: MOT_AV_G.1
- new net MOT_AV_G_OUT-: MOT_AV_G.2
- new net N$10: GRUE.1
- new net N$11: LED4.A, R10.2
- new net N$5: R10.1, RASPPBERRY_PI.31
- new net N$6: GRUE.2
- new net N$9: LIPO.10, LIPO.11, LIPO.12, LIPO.7, LIPO.8, LIPO.9, P1.2
- net +12V: now also ARRET_URGENCE.10, ARRET_URGENCE.11, ARRET_URGENCE.12, ARRET_URGENCE.7, ARRET_URGENCE.8, ARRET_URGENCE.9, AX12_D.DYN_VCC, AX12_G.DYN_VCC, C5.+, C8.+, GRUE.10, GRUE.7, GRUE.8, GRUE.9; no longer ALIM-GRUE.1, LIPO-ET-ARRET-URGENCE.4
- net +3V3: now also R8.1, R9.1, U$3.VIN3V3
- net +5V: now also MOT_AR_D.4, MOT_AR_G.4, MOT_AV_D.4, MOT_AV_G.4, RASPPBERRY_PI.2, RASPPBERRY_PI.4
- net +6V5: now also C6.+, C7.+, XL320_D.DYN_VCC, XL320_G.DYN_VCC
- net GND: now also AX12_D.GND, AX12_G.GND, C10.-, C5.-, C6.-, C7.-, C8.-, GRUE.3, GRUE.4, GRUE.5, GRUE.6, LED4.C, LIPO.1, LIPO.2, LIPO.3, LIPO.4, LIPO.5, LIPO.6, MOT_AR_D.3, MOT_AR_G.3, MOT_AV_D.3, MOT_AV_G.3, RASPPBERRY_PI.14, RASPPBERRY_PI.20, RASPPBERRY_PI.25, RASPPBERRY_PI.30, RASPPBERRY_PI.34, RASPPBERRY_PI.39, RASPPBERRY_PI.6, RASPPBERRY_PI.9, U$2.P$1, U$3.GND, U$3.PWDN, XL320_D.GND, XL320_G.GND; no longer ALIM-GRUE.2, LIPO-ET-ARRET-URGENCE.2
- net N$2: now also R9.2, RASPPBERRY_PI.29, U$2.P$2; no longer LIPO-ET-ARRET-URGENCE.1, P1.2
- net N$3: now also ARRET_URGENCE.1, ARRET_URGENCE.2, ARRET_URGENCE.3, ARRET_URGENCE.4, ARRET_URGENCE.5, ARRET_URGENCE.6, C10.+; no longer LIPO-ET-ARRET-URGENCE.3
- net SERIAL_AX12_5V: now also AX12_D.DATA, AX12_G.DATA
- net SERIAL_XL320_5V: now also XL320_D.DATA, XL320_G.DATA
Other:
- moved on the sheet: ENCODEUR_DROIT, ENCODEUR_GAUCHE, MOT_AR_D, MOT_AR_G, MOT_AV_D, MOT_AV_G, P1, S1

Commit message: pin mapping teensy
Parts:
- added JUMPER: JST-03, con-jst:JST-03
- added LED5, LED6: (no value), led:LEDSMT1206
- added R11: 22k, resistor:R-EU_R0805
- added R12: 6k8, resistor:R-EU_R0805
- added R13, R14: 330, resistor:R-EU_R0805
Connections:
- new net DEL_CLIGNOTANT_D: DELS_ET_TOF_AR.11, PHARES_ET_TOF_AV.9
- new net DEL_CLIGNOTANT_G: DELS_ET_TOF_AR.12, PHARES_ET_TOF_AV.8
- new net DEL_FEUX_NUIT_AR: DELS_ET_TOF_AR.13
- new net DEL_FEUX_NUIT_AV: PHARES_ET_TOF_AV.10
- new net DEL_FEUX_RECUL: DELS_ET_TOF_AR.15
- new net DEL_FEUX_STOP: DELS_ET_TOF_AR.14
- new net DEL_GYRO_1: DEL_GYRO.2
- new net DEL_GYRO_2: DEL_GYRO.3
- new net DEL_GYRO_3: DEL_GYRO.4
- new net DEL_GYRO_4: DEL_GYRO.5
- new net ENC_D_A: ENCODEUR_DROIT.3, U1.18/A4/SDA0
- new net ENC_D_B: ENCODEUR_DROIT.4, U1.39/A20
- new net ENC_G_A: ENCODEUR_GAUCHE.3, U1.16/A2
- new net ENC_G_B: ENCODEUR_GAUCHE.4, U1.17/A3/PWM
- new net GRUE_SERIAL_MISO: GRUE.2, U1.0/RX1/MOSI1
- new net GRUE_SERIAL_MOSI: GRUE.1, U1.1/TX1/MISO1
- new net JUMPER: JUMPER.3, U1.19/A5/SCL0
- new net MOT_AR_D_EN: U1.35/A16/PWM
- new net MOT_AR_D_IN1: U1.36/A17/PWM
- new net MOT_AR_D_IN2: U1.37/A18/SCL1/PWM
- new net MOT_AR_G_EN: U1.21/A7/PWM
- new net MOT_AR_G_IN1: U1.22/A8/PWM
- new net MOT_AR_G_IN2: U1.23/A9/PWM
- new net MOT_AV_D_EN: U1.5/PWM
- new net MOT_AV_D_IN1: U1.6/PWM
- new net MOT_AV_D_IN2: U1.9/RX2/PWM
- new net MOT_AV_G_EN: U1.2/PWM
- new net MOT_AV_G_IN1: U1.3/CAN0-TX/SCL2/PWM
- new net MOT_AV_G_IN2: U1.4/CAN0-RX/SDA2/PWM
- new net N$12: R11.2, R12.1, U1.A21/DAC0
- new net N$13: LED6.A, R14.1
- new net N$14: LED5.A, R13.1
- new net N$15: R13.2, U1.14/A0/PWM
- new net N$16: R14.2, U1.20/A6/PWM
- new net N$19: U2.8/TX3
- new net N$20: U2.11/MOSI
- new net N$21: U2.12/MISO
- new net N$22: U2.14/A1
- new net N$23: U2.15/A1/T
- new net N$24: U2.16/A2/T
- new net N$25: U2.17/A3/T
- new net SCL: DELS_ET_TOF_AR.4, PHARES_ET_TOF_AV.4, U2.19/A5/T/SCL0
- new net SDA: DELS_ET_TOF_AR.3, PHARES_ET_TOF_AV.3, U2.18/A4/T/SDA0
- new net TOF_AR_D: DELS_ET_TOF_AR.7
- new net TOF_AR_G: DELS_ET_TOF_AR.8
- new net TOF_AV: PHARES_ET_TOF_AV.6
- new net TOF_AV_D: PHARES_ET_TOF_AV.7, U2.7/RX3
- new net TOF_AV_G: PHARES_ET_TOF_AV.5, U2.2
- new net TOF_FLAN_AR_D: DELS_ET_TOF_AR.6
- new net TOF_FLAN_AR_G: DELS_ET_TOF_AR.9
- new net TOF_FLAN_AV_D: DELS_ET_TOF_AR.5
- new net TOF_FLAN_AV_G: DELS_ET_TOF_AR.10
- net +12V: now also R11.1
- net +3V3: now also DELS_ET_TOF_AR.2, JUMPER.2, PHARES_ET_TOF_AV.2, U1.3.3V, U2.3.3V
- net +5V: now also ENCODEUR_DROIT.1, ENCODEUR_GAUCHE.1
- net CHOOSE_COLOR: now also U1.A22/DAC1
- net ENC_AR_D_A: now also U1.30/PWM
- net ENC_AR_D_B: now also U1.38/A19/SDA1/PWM
- net ENC_AR_G_A: now also U1.28
- net ENC_AR_G_B: now also U1.29/PWM
- net ENC_AV_D_A: now also U1.26
- net ENC_AV_D_B: now also U1.27
- net ENC_AV_G_A: now also U1.24
- net ENC_AV_G_B: now also U1.25
- net ETH_MISO: now also U1.12/MISO0
- net ETH_MOSI: now also U1.11/MOSI0
- net ETH_RST: now also U1.15/A1
- net ETH_SCLK: now also U1.13/SCK0/LED
- net ETH_SS: now also U1.10/TX2/PWM
- net GND: now also DELS_ET_TOF_AR.1, DEL_GYRO.1, ENCODEUR_DROIT.2, ENCODEUR_GAUCHE.2, JUMPER.1, LED5.C, LED6.C, PHARES_ET_TOF_AV.1, R12.2, U1.AGND, U1.GND, U2.AGND, U2.GND
- net N$10: now also U1.34/A15/RX5, U2.1/TX1/T; no longer GRUE.1
- net N$6: now also U1.33/A14/TX5, U2.0/RX1/T; no longer GRUE.2
- net SERIAL_AX12: now also U1.7/RX3/PWM, U1.8/TX3/PWM
- net SERIAL_XL320: now also U1.31/A12/RX4, U1.32/A13/TX4/SCK1
Other:
- moved on the sheet: DELS_ET_TOF_AR, DEL_GYRO, ENCODEUR_DROIT, ENCODEUR_GAUCHE, PHARES_ET_TOF_AV

Commit message: Début de routage...
Parts:
- added R15, R17, R20, R22, R24, R26, R28, R30, R32, R34: 0, resistor:R-EU_R0805
- added R16, R18, R19, R21, R23, R25, R27, R29, R31, R33: 270, resistor:R-EU_R0805
- added T1, T10, T2, T3, T4, T5, T6, T7, T8, T9: (no value), transistor:BC817-16-NPN-SOT23-BEC
- C1, C2, C3, C4: value (none) -> 10µF
- C10: value (none) -> 4700µF
- LED1, LED5: value (none) -> blue
- LED2: value (none) -> green
- LED3: value (none) -> orange
- LED4, LED6: value (none) -> red
Connections:
- removed net N$19: U2.8/TX3
- removed net N$20: U2.11/MOSI
- removed net N$23: U2.15/A1/T
- removed net N$24: U2.16/A2/T
- new net DEL_CLIGNOTANT_D_PWM: R27.1, U2.20/A6/PWM
- new net DEL_CLIGNOTANT_G_PWM: R25.1, U2.10/TX2/PWM
- new net DEL_FEUX_NUIT_AR_PWM: R29.1, U2.21/A7/PWM
- new net DEL_FEUX_NUIT_AV_PWM: R23.1, U2.9/RX2/PWM
- new net DEL_FEUX_RECUL_PWM: R33.1, U2.23/A9/T/PWM
- new net DEL_FEUX_STOP_PWM: R31.1, U2.22/A8/T/PWM
- new net DEL_GYRO_1_PWM: R19.1, U2.3/CAN-TX/PWM
- new net DEL_GYRO_2_PWM: R16.1, U2.4/CAN-RX/PWM
- new net DEL_GYRO_3_PWM: R18.1, U2.5/PWM
- new net DEL_GYRO_4_PWM: R21.1, U2.6/PWM
- new net N$17: R15.1, T3.E
- new net N$18: R19.2, T3.B
- new net N$26: R18.2, T2.B
- new net N$29: R22.1, T4.E
- new net N$30: R21.2, T4.B
- new net N$33: R24.1, T5.E
- new net N$34: R23.2, T5.B
- new net N$37: R26.1, T6.E
- new net N$38: R25.2, T6.B
- new net N$41: R28.1, T7.E
- new net N$42: R27.2, T7.B
- new net N$45: R30.1, T8.E
- new net N$46: R29.2, T8.B
- new net N$49: R32.1, T9.E
- new net N$50: R31.2, T9.B
- new net N$53: R34.1, T10.E
- new net N$54: R33.2, T10.B
- net +3V3_LEDS: now also T1.C, T10.C, T2.C, T3.C, T4.C, T5.C, T6.C, T7.C, T8.C, T9.C
- net DEL_CLIGNOTANT_D: now also R28.2
- net DEL_CLIGNOTANT_G: now also R26.2
- net DEL_FEUX_NUIT_AR: now also R30.2
- net DEL_FEUX_NUIT_AV: now also R24.2
- net DEL_FEUX_RECUL: now also R34.2
- net DEL_FEUX_STOP: now also R32.2
- net DEL_GYRO_1: now also R15.2
- net DEL_GYRO_2: now also R17.2
- net DEL_GYRO_3: now also R20.2
- net DEL_GYRO_4: now also R22.2
- net GND: now also S1.B, S1.B1
- net N$21: now also R17.1, T1.E; no longer U2.12/MISO
- net N$22: now also R16.2, T1.B; no longer U2.14/A1
- net N$25: now also R20.1, T2.E; no longer U2.17/A3/T
- net TOF_AR_D: now also U2.14/A1
- net TOF_AR_G: now also U2.15/A1/T
- net TOF_AV: now also U2.7/RX3
- net TOF_AV_D: now also U2.8/TX3; no longer U2.7/RX3
- net TOF_FLAN_AR_D: now also U2.12/MISO
- net TOF_FLAN_AR_G: now also U2.16/A2/T
- net TOF_FLAN_AV_D: now also U2.11/MOSI
- net TOF_FLAN_AV_G: now also U2.17/A3/T
Other:
- moved on the sheet: DELS_ET_TOF_AR, DEL_GYRO, ENCODEUR_DROIT, ENCODEUR_GAUCHE, GRUE, JUMPER, LED1, MOT_AR_D, MOT_AR_G, MOT_AV_D, MOT_AV_G, PHARES_ET_TOF_AV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
