File: electronique/camion-grue.sch (EAGLE design)
At the start: 91 parts, among them P1 RGEF800, Q1 BSS138, Q2 BSS138, U1 TEENSY_3.5_DIL+USB, U2 TEENSY_3.1-3.2_DIL

Commit message: ajout carte elec grue
Parts:
- C1, C2, C3, C4: device resistor:CPOL-EUE2.5-7 -> resistor:C-EUC0805
- C5, C6, C7, C8: device resistor:CPOL-EUE2.5-6 -> resistor:C-EUC0805
Connections:
- net +12V: now also C1.1, C2.1, C4.1, C5.1, C8.1; no longer C1.+, C2.+, C4.+, C5.+, C8.+
- net +6V5: now also C6.1, C7.1; no longer C6.+, C7.+
- net 12V_AUX: now also C3.1; no longer C3.+
- net GND: now also C1.2, C2.2, C3.2, C4.2, C5.2, C6.2, C7.2, C8.2; no longer C1.-, C2.-, C3.-, C4.-, C5.-, C6.-, C7.-, C8.-
Changed lines of the file:
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@@
 <part name="DC3" library="dc-dc-converter" library_urn="urn:adsk.eagle:library:208" deviceset="R-78C*-1.0" device="" package3d_urn="urn:adsk.eagle:package:12318/1" technology="5.0"/>
 <part name="DC4" library="dc-dc-converter" library_urn="urn:adsk.eagle:library:208" deviceset="R-78C*-1.0" device="" package3d_urn="urn:adsk.eagle:package:12318/1" technology="9.0"/>
-<part name="C1" library="resistor" library_urn="urn:adsk.eagle:library:348" deviceset="CPOL-EU" device="E2.5-7" package3d_urn="urn:adsk.eagle:package:25830/1" value="10µF"/>
-<part name="C2" library="resistor" library_urn="urn:adsk.eagle:library:348" deviceset="CPOL-EU" device="E2.5-7" package3d_urn="urn:adsk.eagle:package:25830/1" value="10µF"/>
-<part name="C3" library="resistor" library_urn="urn:adsk.eagle:library:348" deviceset="CPOL-EU" device="E2.5-7" package3d_urn="urn:adsk.eagle:package:25830/1" value="10µF"/>
-<part name="C4" library="resistor" library_urn="urn:adsk.eagle:library:348" deviceset="CPOL-EU" device="E2.5-7" package3d_urn="urn:adsk.eagle:package:25830/1" value="10µF"/>
+<part name="C1" library="resistor" library_urn="urn:adsk.eagle:library:348" deviceset="C-EU" device="C0805" package3d_urn="urn:adsk.eagle:package:26137/1" value="10µF"/>
+<part name="C2" library="resistor" library_urn="urn:adsk.eagle:library:348" deviceset="C-EU" device="C0805" package3d_urn="urn:adsk.eagle:package:26137/1" value="10µF"/>
+<part name="C3" library="resistor" library_urn="urn:adsk.eagle:library:348" deviceset="C-EU" device="C0805" package3d_urn="urn:adsk.eagle:package:26137/1" value="10µF"/>
+<part name="C4" library="resistor" library_urn="urn:adsk.eagle:library:348" deviceset="C-EU" device="C0805" package3d_urn="urn:adsk.eagle:package:26137/1" value="10µF"/>
 <part name="SUPPLY13" library="supply2" library_urn="urn:adsk.eagle:library:372" deviceset="GND" device=""/>
 <part name="SUPPLY14" library="supply2" library_urn="urn:adsk.eagle:library:372" deviceset="+12V" device=""/>
@@
 <part name="AX12_G" library="1NTech_pinhead" deviceset="DYNAMIXEL-1X03" device="AX"/>
 <part name="XL320_G" library="1NTech_pinhead" deviceset="DYNAMIXEL-1X03" device="XL"/>
-<part name="C5" library="resistor" library_urn="urn:adsk.eagle:library:348" deviceset="CPOL-EU" device="E2.5-6" package3d_urn="urn:adsk.eagle:package:25832/1" value="1µF"/>
-<part name="C7" library="resistor" library_urn="urn:adsk.eagle:library:348" deviceset="CPOL-EU" device="E2.5-6" package3d_urn="urn:adsk.eagle:package:25832/1" value="1µF"/>
+<part name="C5" library="resistor" library_urn="urn:adsk.eagle:library:348" deviceset="C-EU" device="C0805" package3d_urn="urn:adsk.eagle:package:26137/1" value="1µF"/>
+<part name="C7" library="resistor" library_urn="urn:adsk.eagle:library:348" deviceset="C-EU" device="C0805" package3d_urn="urn:adsk.eagle:package:26137/1" value="1µF"/>
 <part name="SUPPLY29" library="supply2" library_urn="urn:adsk.eagle:library:372" deviceset="GND" device=""/>
 <part name="SUPPLY31" library="supply2" library_urn="urn:adsk.eagle:library:372" deviceset="GND" device=""/>
 <part name="SUPPLY30" library="supply2" library_urn="urn:adsk.eagle:library:372" deviceset="+12V" device=""/>
 <part name="XL320_D" library="1NTech_pinhead" deviceset="DYNAMIXEL-1X03" device="XL"/>
-<part name="C6" library="resistor" library_urn="urn:adsk.eagle:library:348" deviceset="CPOL-EU" device="E2.5-6" package3d_urn="urn:adsk.eagle:package:25832/1" value="1µF"/>
+<part name="C6" library="resistor" library_urn="urn:adsk.eagle:library:348" deviceset="C-EU" device="C0805" package3d_urn="urn:adsk.eagle:package:26137/1" value="1µF"/>
 <part name="SUPPLY32" library="supply2" library_urn="urn:adsk.eagle:library:372" deviceset="GND" device=""/>
 <part name="AX12_D" library="1NTech_pinhead" deviceset="DYNAMIXEL-1X03" device="AX"/>
-<part name="C8" library="resistor" library_urn="urn:adsk.eagle:library:348" deviceset="CPOL-EU" device="E2.5-6" package3d_urn="urn:adsk.eagle:package:25832/1" value="1µF"/>
+<part name="C8" library="resistor" library_urn="urn:adsk.eagle:library:348" deviceset="C-EU" device="C0805" package3d_urn="urn:adsk.eagle:package:26137/1" value="1µF"/>
 <part name="SUPPLY33" library="supply2" library_urn="urn:adsk.eagle:library:372" deviceset="GND" device=""/>
 <part name="SUPPLY34" library="supply2" library_urn="urn:adsk.eagle:library:372" deviceset="+12V" device=""/>
@@
 <segment>
 <pinref part="DC1" gate="G$1" pin="VIN"/>
-<pinref part="C1" gate="G$1" pin="+"/>
+<pinref part="C1" gate="G$1" pin="1"/>
 <wire x1="96.52" y1="241.3" x2="93.98" y2="241.3" width="0.1524" layer="91"/>
 <wire x1="93.98" y1="241.3" x2="93.98" y2="238.76" width="0.1524" layer="91"/>
@@
 <pinref part="DC2" gate="G$1" pin="VIN"/>
 <wire x1="91.44" y1="215.9" x2="93.98" y2="215.9" width="0.1524" layer="91"/>
-<pinref part="C2" gate="G$1" pin="+"/>
+<pinref part="C2" gate="G$1" pin="1"/>
 <wire x1="93.98" y1="215.9" x2="96.52" y2="215.9" width="0.1524" layer="91"/>
 <wire x1="93.98" y1="213.36" x2="93.98" y2="215.9" width="0.1524" layer="91"/>
@@
 </segment>
 <segment>
-<pinref part="C4" gate="G$1" pin="+"/>
+<pinref part="C4" gate="G$1" pin="1"/>
 <pinref part="DC4" gate="G$1" pin="VIN"/>
 <wire x1="93.98" y1="162.56" x2="93.98" y2="165.1" width="0.1524" layer="91"/>
@@
 <segment>
 <pinref part="AX12_G" gate="G$1" pin="DYN_VCC"/>
-<pinref part="C5" gate="G$1" pin="+"/>
+<pinref part="C5" gate="G$1" pin="1"/>
 <wire x1="86.36" y1="48.26" x2="86.36" y2="58.42" width="0.1524" layer="91"/>
 <pinref part="SUPPLY30" gate="+12V" pin="+12V"/>
@@
 <segment>
 <pinref part="AX12_D" gate="G$1" pin="DYN_VCC"/>
-<pinref part="C8" gate="G$1" pin="+"/>
+<pinref part="C8" gate="G$1" pin="1"/>
 <wire x1="111.76" y1="48.26" x2="111.76" y2="58.42" width="0.1524" layer="91"/>
 <pinref part="SUPPLY34" gate="+12V" pin="+12V"/>
@@
 </segment>
 <segment>
-<pinref part="C1" gate="G$1" pin="-"/>
+<pinref part="C1" gate="G$1" pin="2"/>
 <pinref part="DC1" gate="G$1" pin="GND"/>
 <wire x1="93.98" y1="231.14" x2="109.22" y2="231.14" width="0.1524" layer="91"/>
@@
 </segment>
 <segment>
-<pinref part="C2" gate="G$1" pin="-"/>
+<pinref part="C2" gate="G$1" pin="2"/>
 <pinref part="DC2" gate="G$1" pin="GND"/>
 <wire x1="93.98" y1="205.74" x2="109.22" y2="205.74" width="0.1524" layer="91"/>
@@
 </segment>
 <segment>
-<pinref part="C3" gate="G$1" pin="-"/>
+<pinref part="C3" gate="G$1" pin="2"/>
 <pinref part="SUPPLY17" gate="GND" pin="GND"/>
 <wire x1="93.98" y1="180.34" x2="109.22" y2="180.34" width="0.1524" layer="91"/>
@@
 </segment>
 <segment>
-<pinref part="C4" gate="G$1" pin="-"/>
+<pinref part="C4" gate="G$1" pin="2"/>
 <pinref part="DC4" gate="G$1" pin="GND"/>
 <wire x1="93.98" y1="154.94" x2="109.22" y2="154.94" width="0.1524" layer="91"/>
@@
 <pinref part="AX12_G" gate="G$1" pin="GND"/>
 <wire x1="91.44" y1="48.26" x2="91.44" y2="53.34" width="0.1524" layer="91"/>
-<pinref part="C5" gate="G$1" pin="-"/>
+<pinref part="C5" gate="G$1" pin="2"/>
 <wire x1="91.44" y1="53.34" x2="93.98" y2="53.34" width="0.1524" layer="91"/>
 <wire x1="93.98" y1="53.34" x2="93.98" y2="58.42" width="0.1524" layer="91"/>
@@
 </segment>
 <segment>
-<pinref part="C7" gate="G$1" pin="-"/>
+<pinref part="C7" gate="G$1" pin="2"/>
 <pinref part="SUPPLY31" gate="GND" pin="GND"/>
 <wire x1="96.52" y1="25.4" x2="93.98" y2="25.4" width="0.1524" layer="91"/>
@@
 </segment>
 <segment>
-<pinref part="C6" gate="G$1" pin="-"/>
+<pinref part="C6" gate="G$1" pin="2"/>
 <pinref part="SUPPLY32" gate="GND" pin="GND"/>
 <wire x1="121.92" y1="25.4" x2="119.38" y2="25.4" width="0.1524" layer="91"/>
@@
 <pinref part="AX12_D" gate="G$1" pin="GND"/>
 <wire x1="116.84" y1="48.26" x2="116.84" y2="53.34" width="0.1524" layer="91"/>
-<pinref part="C8" gate="G$1" pin="-"/>
+<pinref part="C8" gate="G$1" pin="2"/>
 <wire x1="116.84" y1="53.34" x2="119.38" y2="53.34" width="0.1524" layer="91"/>
 <wire x1="119.38" y1="53.34" x2="119.38" y2="58.42" width="0.1524" layer="91"/>
@@
 <net name="12V_AUX" class="0">
 <segment>
-<pinref part="C3" gate="G$1" pin="+"/>
+<pinref part="C3" gate="G$1" pin="1"/>
 <pinref part="DC3" gate="G$1" pin="VIN"/>
 <wire x1="93.98" y1="187.96" x2="93.98" y2="190.5" width="0.1524" layer="91"/>
@@
 <segment>
 <pinref part="XL320_G" gate="G$1" pin="DYN_VCC"/>
-<pinref part="C7" gate="G$1" pin="+"/>
+<pinref part="C7" gate="G$1" pin="1"/>
 <wire x1="86.36" y1="15.24" x2="86.36" y2="25.4" width="0.1524" layer="91"/>
 <wire x1="86.36" y1="25.4" x2="86.36" y2="30.48" width="0.1524" layer="91"/>
@@
 <segment>
 <pinref part="XL320_D" gate="G$1" pin="DYN_VCC"/>
-<pinref part="C6" gate="G$1" pin="+"/>
+<pinref part="C6" gate="G$1" pin="1"/>
 <wire x1="111.76" y1="15.24" x2="111.76" y2="25.4" width="0.1524" layer="91"/>
 <wire x1="111.76" y1="25.4" x2="111.76" y2="30.48" width="0.1524" layer="91"/>
