File: electronique/camion-grue.sch (EAGLE design)
At the start: 92 parts, among them P1 RGEF800, Q1 BSS138, Q2 BSS138, U1 TEENSY_3.5_DIL+USB, U2 TEENSY_3.1-3.2_DIL

Commit message: Elec robot: régulateur 5V dédié pour la logique, indépendant de celui de la RPI
Parts:
- added C11: 22µF, resistor:C-EUC0805
- added C9: 10µF, resistor:C-EUC0805
- added IC3: REG1117, burr-brown:REG1117
Connections:
- new net +5V_RPI: DC3.VOUT, R1.2, RASPPBERRY_PI.2, RASPPBERRY_PI.4
- net +12V: now also C9.1, IC3.VIN
- net +5V: now also C11.1, IC3.VOUT; no longer DC3.VOUT, R1.2, RASPPBERRY_PI.2, RASPPBERRY_PI.4
- net GND: now also C11.2, C9.2, IC3.GND
Changed lines of the file:
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@@
 <?xml version="1.0" encoding="utf-8"?>
 <!DOCTYPE eagle SYSTEM "eagle.dtd">
-<eagle version="8.5.1">
+<eagle version="8.6.0">
 <drawing>
 <settings>
@@
 <part name="SUPPLY16" library="supply2" library_urn="urn:adsk.eagle:library:372" deviceset="GND" device=""/>
 <part name="SUPPLY17" library="supply2" library_urn="urn:adsk.eagle:library:372" deviceset="GND" device=""/>
-<part name="SUPPLY18" library="supply2" library_urn="urn:adsk.eagle:library:372" deviceset="+5V" device=""/>
 <part name="SUPPLY19" library="supply2" library_urn="urn:adsk.eagle:library:372" deviceset="GND" device=""/>
 <part name="SUPPLY20" library="supply2" library_urn="urn:adsk.eagle:library:372" deviceset="+12V" device=""/>
@@
 <part name="SUPPLY45" library="supply2" library_urn="urn:adsk.eagle:library:372" deviceset="GND" device=""/>
 <part name="U$2" library="push-button" deviceset="PUSH-BUTTON" device=""/>
-<part name="SUPPLY46" library="supply2" library_urn="urn:adsk.eagle:library:372" deviceset="+5V" device=""/>
 <part name="SUPPLY47" library="supply2" library_urn="urn:adsk.eagle:library:372" deviceset="GND" device=""/>
 <part name="SUPPLY48" library="supply2" library_urn="urn:adsk.eagle:library:372" deviceset="GND" device=""/>
@@
 <part name="USB_BACKUP_DEBUG" library="pinhead" library_urn="urn:adsk.eagle:library:325" deviceset="PINHD-1X3" device="" package3d_urn="urn:adsk.eagle:package:22458/2"/>
 <part name="SUPPLY73" library="supply2" library_urn="urn:adsk.eagle:library:372" deviceset="GND" device=""/>
+<part name="SUPPLY74" library="supply2" library_urn="urn:adsk.eagle:library:372" deviceset="+12V" device=""/>
+<part name="SUPPLY75" library="supply2" library_urn="urn:adsk.eagle:library:372" deviceset="+5V" device=""/>
+<part name="SUPPLY76" library="supply2" library_urn="urn:adsk.eagle:library:372" deviceset="GND" device=""/>
+<part name="IC3" library="burr-brown" library_urn="urn:adsk.eagle:library:111" deviceset="REG1117" device="" package3d_urn="urn:adsk.eagle:package:4940/1">
+<attribute name="RS" value="885-5432"/>
+</part>
+<part name="C9" library="resistor" library_urn="urn:adsk.eagle:library:348" deviceset="C-EU" device="C0805" package3d_urn="urn:adsk.eagle:package:26137/1" value="10µF"/>
+<part name="C11" library="resistor" library_urn="urn:adsk.eagle:library:348" deviceset="C-EU" device="C0805" package3d_urn="urn:adsk.eagle:package:26137/1" value="22µF"/>
 </parts>
 <sheets>
@@
 <instance part="SUPPLY16" gate="GND" x="109.22" y="203.2"/>
 <instance part="SUPPLY17" gate="GND" x="109.22" y="177.8"/>
-<instance part="SUPPLY18" gate="+5V" x="127" y="190.5" rot="R270"/>
 <instance part="SUPPLY19" gate="GND" x="109.22" y="152.4"/>
 <instance part="SUPPLY20" gate="+12V" x="88.9" y="165.1" rot="R90"/>
@@
 <instance part="SUPPLY45" gate="GND" x="109.22" y="101.6" rot="R90"/>
 <instance part="U$2" gate="G$1" x="220.98" y="25.4"/>
-<instance part="SUPPLY46" gate="+5V" x="259.08" y="60.96" rot="R270"/>
 <instance part="SUPPLY47" gate="GND" x="259.08" y="55.88" rot="R90"/>
 <instance part="SUPPLY48" gate="GND" x="259.08" y="45.72" rot="R90"/>
@@
 <instance part="USB_BACKUP_DEBUG" gate="A" x="340.36" y="35.56"/>
 <instance part="SUPPLY73" gate="GND" x="330.2" y="40.64" rot="R180"/>
+<instance part="SUPPLY74" gate="+12V" x="144.78" y="81.28"/>
+<instance part="SUPPLY75" gate="+5V" x="175.26" y="81.28"/>
+<instance part="SUPPLY76" gate="GND" x="160.02" y="60.96"/>
+<instance part="IC3" gate="G$1" x="160.02" y="78.74">
+<attribute name="RS" x="160.02" y="78.74" size="1.778" layer="96" display="off"/>
+</instance>
+<instance part="C9" gate="G$1" x="144.78" y="73.66"/>
+<instance part="C11" gate="G$1" x="175.26" y="73.66"/>
 </instances>
 <busses>
@@
 </segment>
 <segment>
-<pinref part="DC3" gate="G$1" pin="VOUT"/>
-<wire x1="121.92" y1="190.5" x2="124.46" y2="190.5" width="0.1524" layer="91"/>
-<pinref part="SUPPLY18" gate="+5V" pin="+5V"/>
-<pinref part="R1" gate="G$1" pin="2"/>
-<wire x1="121.92" y1="190.5" x2="121.92" y2="185.42" width="0.1524" layer="91"/>
-<wire x1="121.92" y1="185.42" x2="124.46" y2="185.42" width="0.1524" layer="91"/>
-<junction x="121.92" y="190.5"/>
-</segment>
-<segment>
 <pinref part="R3" gate="G$1" pin="1"/>
 <wire x1="50.8" y1="58.42" x2="50.8" y2="60.96" width="0.1524" layer="91"/>
@@
 </segment>
 <segment>
-<pinref part="RASPPBERRY_PI" gate="A" pin="2"/>
-<wire x1="251.46" y1="60.96" x2="256.54" y2="60.96" width="0.1524" layer="91"/>
-<pinref part="RASPPBERRY_PI" gate="A" pin="4"/>
-<wire x1="251.46" y1="58.42" x2="256.54" y2="58.42" width="0.1524" layer="91"/>
-<wire x1="256.54" y1="58.42" x2="256.54" y2="60.96" width="0.1524" layer="91"/>
-<pinref part="SUPPLY46" gate="+5V" pin="+5V"/>
-<junction x="256.54" y="60.96"/>
-</segment>
-<segment>
 <pinref part="ENCODEUR_GAUCHE" gate="G$1" pin="1"/>
 <pinref part="SUPPLY56" gate="+5V" pin="+5V"/>
@@
 <pinref part="SUPPLY59" gate="+5V" pin="+5V"/>
 <wire x1="205.74" y1="177.8" x2="208.28" y2="177.8" width="0.1524" layer="91"/>
+</segment>
+<segment>
+<pinref part="IC3" gate="G$1" pin="VOUT"/>
+<pinref part="SUPPLY75" gate="+5V" pin="+5V"/>
+<wire x1="175.26" y1="78.74" x2="172.72" y2="78.74" width="0.1524" layer="91"/>
+<pinref part="C11" gate="G$1" pin="1"/>
+<wire x1="175.26" y1="76.2" x2="175.26" y2="78.74" width="0.1524" layer="91"/>
+<junction x="175.26" y="78.74"/>
 </segment>
 </net>
@@
 <wire x1="375.92" y1="172.72" x2="375.92" y2="175.26" width="0.1524" layer="91"/>
 </segment>
+<segment>
+<pinref part="IC3" gate="G$1" pin="VIN"/>
+<pinref part="SUPPLY74" gate="+12V" pin="+12V"/>
+<wire x1="144.78" y1="78.74" x2="147.32" y2="78.74" width="0.1524" layer="91"/>
+<pinref part="C9" gate="G$1" pin="1"/>
+<wire x1="144.78" y1="76.2" x2="144.78" y2="78.74" width="0.1524" layer="91"/>
+<junction x="144.78" y="78.74"/>
+</segment>
 </net>
 <net name="GND" class="0">
@@
 <wire x1="337.82" y1="38.1" x2="330.2" y2="38.1" width="0.1524" layer="91"/>
 <pinref part="SUPPLY73" gate="GND" pin="GND"/>
+</segment>
+<segment>
+<pinref part="SUPPLY76" gate="GND" pin="GND"/>
+<pinref part="IC3" gate="G$1" pin="GND"/>
+<wire x1="160.02" y1="63.5" x2="160.02" y2="66.04" width="0.1524" layer="91"/>
+<pinref part="C9" gate="G$1" pin="2"/>
+<wire x1="144.78" y1="68.58" x2="144.78" y2="66.04" width="0.1524" layer="91"/>
+<wire x1="144.78" y1="66.04" x2="160.02" y2="66.04" width="0.1524" layer="91"/>
+<junction x="160.02" y="66.04"/>
+<pinref part="C11" gate="G$1" pin="2"/>
+<wire x1="175.26" y1="68.58" x2="175.26" y2="66.04" width="0.1524" layer="91"/>
+<wire x1="175.26" y1="66.04" x2="160.02" y2="66.04" width="0.1524" layer="91"/>
 </segment>
 </net>
@@
 </segment>
 </net>
+<net name="+5V_RPI" class="0">
+<segment>
+<pinref part="RASPPBERRY_PI" gate="A" pin="2"/>
+<wire x1="251.46" y1="60.96" x2="256.54" y2="60.96" width="0.1524" layer="91"/>
+<pinref part="RASPPBERRY_PI" gate="A" pin="4"/>
+<wire x1="251.46" y1="58.42" x2="256.54" y2="58.42" width="0.1524" layer="91"/>
+<wire x1="256.54" y1="58.42" x2="256.54" y2="60.96" width="0.1524" layer="91"/>
+<wire x1="256.54" y1="60.96" x2="259.08" y2="60.96" width="0.1524" layer="91"/>
+<junction x="256.54" y="60.96"/>
+<label x="259.08" y="60.96" size="1.27" layer="95" xref="yes"/>
+</segment>
+<segment>
+<pinref part="DC3" gate="G$1" pin="VOUT"/>
+<wire x1="121.92" y1="190.5" x2="124.46" y2="190.5" width="0.1524" layer="91"/>
+<pinref part="R1" gate="G$1" pin="2"/>
+<wire x1="121.92" y1="190.5" x2="121.92" y2="185.42" width="0.1524" layer="91"/>
+<wire x1="121.92" y1="185.42" x2="124.46" y2="185.42" width="0.1524" layer="91"/>
+<junction x="121.92" y="190.5"/>
+<label x="124.46" y="190.5" size="1.27" layer="95" xref="yes"/>
+</segment>
+</net>
