File: electronique/grue.brd (EAGLE design)
At the start: 90.5 x 48.5 mm, 65 parts, among them IC3 REG1117, Q1 BSS138, Q2 BSS138

Commit message: Elec version finale + Ajout fichiers gerber
Other:
- board text added: "GYRO"
- board text added: "M"
- board text added: "TOF LPD"
- board text added: "TOF LPG"
- board text added: "TOF PINCE"
Changed lines of the file:
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@@
 <?xml version="1.0" encoding="utf-8"?>
 <!DOCTYPE eagle SYSTEM "eagle.dtd">
-<eagle version="8.5.1">
+<eagle version="8.6.0">
 <drawing>
 <settings>
@@
 <layer number="21" name="tPlace" color="7" fill="1" visible="yes" active="yes"/>
 <layer number="22" name="bPlace" color="7" fill="1" visible="yes" active="yes"/>
-<layer number="23" name="tOrigins" color="15" fill="1" visible="yes" active="yes"/>
-<layer number="24" name="bOrigins" color="15" fill="1" visible="yes" active="yes"/>
-<layer number="25" name="tNames" color="7" fill="1" visible="yes" active="yes"/>
-<layer number="26" name="bNames" color="7" fill="1" visible="yes" active="yes"/>
+<layer number="23" name="tOrigins" color="15" fill="1" visible="no" active="yes"/>
+<layer number="24" name="bOrigins" color="15" fill="1" visible="no" active="yes"/>
+<layer number="25" name="tNames" color="7" fill="1" visible="no" active="yes"/>
+<layer number="26" name="bNames" color="7" fill="1" visible="no" active="yes"/>
 <layer number="27" name="tValues" color="7" fill="1" visible="no" active="yes"/>
 <layer number="28" name="bValues" color="7" fill="1" visible="no" active="yes"/>
@@
 <layer number="37" name="tTest" color="7" fill="1" visible="no" active="yes"/>
 <layer number="38" name="bTest" color="7" fill="1" visible="no" active="yes"/>
-<layer number="39" name="tKeepout" color="4" fill="11" visible="yes" active="yes"/>
-<layer number="40" name="bKeepout" color="1" fill="11" visible="yes" active="yes"/>
-<layer number="41" name="tRestrict" color="4" fill="10" visible="yes" active="yes"/>
-<layer number="42" name="bRestrict" color="1" fill="10" visible="yes" active="yes"/>
-<layer number="43" name="vRestrict" color="2" fill="10" visible="yes" active="yes"/>
+<layer number="39" name="tKeepout" color="4" fill="11" visible="no" active="yes"/>
+<layer number="40" name="bKeepout" color="1" fill="11" visible="no" active="yes"/>
+<layer number="41" name="tRestrict" color="4" fill="10" visible="no" active="yes"/>
+<layer number="42" name="bRestrict" color="1" fill="10" visible="no" active="yes"/>
+<layer number="43" name="vRestrict" color="2" fill="10" visible="no" active="yes"/>
 <layer number="44" name="Drills" color="7" fill="1" visible="no" active="yes"/>
 <layer number="45" name="Holes" color="7" fill="1" visible="yes" active="yes"/>
@@
 <wire x1="58.3" y1="40.7" x2="58.3" y2="22.5" width="0.2" layer="21"/>
 <wire x1="58.3" y1="22.5" x2="52.3" y2="16.5" width="0.2" layer="21"/>
+<text x="14.9" y="38.4" size="2.54" layer="51" align="center">M</text>
+<rectangle x1="12.4" y1="40" x2="17.4" y2="46.4" layer="51"/>
+<wire x1="12.6" y1="40.2" x2="12.6" y2="36.6" width="0.4" layer="51"/>
+<wire x1="12.6" y1="36.6" x2="13" y2="36.6" width="0.4" layer="51"/>
+<wire x1="13" y1="36.6" x2="16.8" y2="36.6" width="0.4" layer="51"/>
+<wire x1="16.8" y1="36.6" x2="17.2" y2="36.6" width="0.4" layer="51"/>
+<wire x1="17.2" y1="36.6" x2="17.2" y2="40.2" width="0.4" layer="51"/>
+<wire x1="13" y1="40.2" x2="13" y2="36.6" width="0.4" layer="51"/>
+<wire x1="16.8" y1="40.2" x2="16.8" y2="36.6" width="0.4" layer="51"/>
+<text x="26" y="9" size="1.778" layer="51" align="top-center">GYRO</text>
+<text x="82.6" y="13.9" size="1.778" layer="51" rot="SR270" align="top-center">TOF LPG</text>
+<text x="34.8" y="16" size="1.778" layer="51" rot="SR0" align="top-center">TOF LPD</text>
+<text x="48.8" y="16" size="1.778" layer="51" rot="SR0" align="top-center">TOF PINCE</text>
 </plain>
 <attributes>
@@
 <wire x1="14.44" y1="37.39" x2="14.55" y2="37.5" width="0.6096" layer="16"/>
 <polygon width="0.2" layer="1">
-<vertex x="-2.2" y="50.4"/>
-<vertex x="92.8" y="50.4"/>
-<vertex x="92.8" y="-1.8"/>
-<vertex x="-2.2" y="-1.8"/>
+<vertex x="-0.5" y="48.5"/>
+<vertex x="90" y="48.5"/>
+<vertex x="90" y="0"/>
+<vertex x="-0.5" y="0"/>
 </polygon>
 <polygon width="0.2" layer="16">
-<vertex x="-3" y="51.2"/>
-<vertex x="93.6" y="51.2"/>
-<vertex x="93.6" y="-2.4"/>
-<vertex x="-3" y="-2.4"/>
+<vertex x="-0.5" y="48.5"/>
+<vertex x="90" y="48.5"/>
+<vertex x="90" y="0"/>
+<vertex x="-0.5" y="0"/>
 </polygon>
 <via x="44.4" y="34.2" extent="1-16" drill="0.35"/>
