File: electronique/intech-senpai-camion-grue-complet.brd (EAGLE design)
At the start: 129 x 106 mm, 135 parts, among them IC3 REG1117, P1 RGEF800, Q1 BSS138, Q2 BSS138, U1 TEENSY_3.5_DIL+USB, U2 TEENSY_3.1-3.2_DIL

Commit message: Elec version finale + Ajout fichiers gerber
Parts:
- added AX12_G1: DYNAMIXEL-1X03AX, 1NTech_pinhead:DYNAMIXEL_AX_1X03
- added C12, C13, C17, MULTI-BUTTON-1:C1, MULTI-BUTTON-2:C1: 1µF, resistor:C0805
- added C14, C15, C18, C19, C20: 10µF, resistor:C0805
- added C16: 22µF, resistor:C0805
- added D2, H-BRIDGE1:D1, H-BRIDGE1:D2, H-BRIDGE1:D3, H-BRIDGE1:D4, H-BRIDGE1:D5, H-BRIDGE1:D6, H-BRIDGE1:D7, H-BRIDGE1:D8: S1M, diode:SMA
- added DC-DC-6V: DC-DC-CONVERTER, dc-dc-converter-6v:DC-DC-CONVERTER
- added DC5, DC7: R-78C3.3-1.0, dc-dc-converter:SIP3
- added DC6: R-78C5.0-1.0, dc-dc-converter:SIP3
- added DEBUG_UART, MOT_H, MOT_V: (no value), pinhead:1X06
- added F1: MF-LSMF300, polyswitch:MF-LSMF300
- added F2: MF-MSMF110, polyswitch:MF-MSMF110
- added GRUE1: JST-10, con-jst:GH-10-V
- added GYRO, LIPO1: JST-04GH-V, con-jst:GH-04-V
- added H-BRIDGE1:C1, H-BRIDGE1:C2: 100nF, resistor:C0805
- added H-BRIDGE1:IC1: L298, st-microelectronics:MULTIWATT-15
- added H-BRIDGE1:R1, H-BRIDGE1:R2, H-BRIDGE1:R3, H-BRIDGE1:R4, H-BRIDGE1:R5, H-BRIDGE1:R6, MULTI-BUTTON-1:R3, MULTI-BUTTON-2:R3, R35, R36, R37, R38: 10k, resistor:R0805
- added IC1: REG1117, burr-brown:SOT223
- added LED100, LED117, LED118, LED119, LED120, LED121, LED122, LED123, LED132, LED149, LED150, LED151, LED152, LED153, LED154, LED155, LED34, LED51, LED52, LED53, LED54, LED55, LED56, LED57: jaune, led:LED5MM
- added LED101, LED110, LED111, LED112, LED113, LED114, LED115, LED116, LED133, LED142, LED143, LED144, LED145, LED146, LED147, LED148, LED35, LED44, LED45, LED46, LED47, LED48, LED49, LED50, LED97: vert, led:LED5MM
- added LED102, LED124, LED125, LED126, LED127, LED128, LED129, LED130, LED134, LED156, LED157, LED158, LED159, LED160, LED161, LED162, LED36, LED58, LED59, LED60, LED61, LED62, LED63, LED64, LED98: bleu, led:LED5MM
- added LED103, LED104, LED105, LED106, LED107, LED108, LED109, LED131, LED135, LED136, LED137, LED138, LED139, LED140, LED141, LED33, LED37, LED38, LED39, LED40, LED41, LED42, LED43, LED99: orange, led:LED5MM
- added MULTI-BUTTON-1:R1, MULTI-BUTTON-2:R1: 4k7, resistor:R0805
- added MULTI-BUTTON-1:R2, MULTI-BUTTON-2:R2: 2k2, resistor:R0805
- added MULTI-BUTTON-1:U1, MULTI-BUTTON-1:U2, MULTI-BUTTON-1:U3, MULTI-BUTTON-2:U1, MULTI-BUTTON-2:U2, MULTI-BUTTON-2:U3, U$4: PUSH-BUTTON, push-button:PUSH-BUTTON
- added Q3, Q4: BSS138, transistor-small-signal:SOT23
- added R39, R41, R59, R60, R61, R62, R66, R67, R68, R69, R78, R79, R80, R81: 270, resistor:R0805
- added R40, R42, R46, R47, R48, R49, R50, R51, R52, R53, R54, R55, R56, R57, R58, R63, R64, R65, R70, R71, R72, R73, R74, R75, R76, R77: 0, resistor:R0805
- added R43: 220, resistor:R0805
- added R44, R82: 1k, resistor:R0805
- added R45: 470, resistor:R0805
- added RPI: RPI-ZERO, RPI-Zero:RASPBERRYPI_BASTELSTUBE_V13_RASPI_BOARD_B+_FULL
- added S2: TL36PO, switch:TL3XPO
- added T11, T12, T13, T14, T15, T16, T17, T18, T19, T20, T21, T22, T23, T24: (no value), transistor:SOT23-BEC
- added TOF_LP_D_AND_DISPLAY, TOF_LP_G: JST-05, con-jst:GH-05-V
- added TOF_PINCE: JST-06, con-jst:GH-06-V
- added U$1: TEENSY_3.1-3.2_DIL+4, Teensy_libSG:TEENSY_3.0-3.2&LC_DIL+4
- added XL320_G1, XL320_G2: DYNAMIXEL-1X03XL, 1NTech_pinhead:DYNAMIXEL_XL_1X03
Connections:
- new net +12VB: C18.2, C19.2, DC6.1, DC7.1, S2.1
- new net +12VG: AX12_G1.DYN_VCC, C12.1, C14.1, C15.1, DC-DC-6V.VIN, DC5.1, GRUE1.10, GRUE1.7, GRUE1.8, GRUE1.9, IC1.3
- new net +3V3G: DC5.3, MULTI-BUTTON-1:R1.1, MULTI-BUTTON-2:R1.1, Q3.1, Q4.1, R35.1, R37.1, T11.C, T12.C, TOF_LP_D_AND_DISPLAY.2, TOF_LP_G.2, TOF_PINCE.2, U$1.3.3V
- new net +5VB: DC6.3, R44.1, RPI.2, RPI.4
- new net +5VG: C16.1, H-BRIDGE1:C2.2, H-BRIDGE1:IC1.9, IC1.2, MOT_H.4, MOT_V.4, R36.1, R38.1
- new net +6V: C13.1, C17.1, DC-DC-6V.VOUT, F1.2, XL320_G1.VCC, XL320_G2.VCC
- new net 3V3@1: R82.1, RPI.1
- new net AREF: U$1.AREF
- new net DEL_BLEU_1: LED134.A, LED156.A, LED157.A, LED158.A, LED159.A, LED160.A, LED161.A, LED162.A, T20.E
- new net DEL_BLEU_1_PWM: R62.2, RPI.36
- new net DEL_BLEU_2: LED36.A, LED58.A, LED59.A, LED60.A, LED61.A, LED62.A, LED63.A, LED64.A, T16.E
- new net DEL_BLEU_2_PWM: R69.2, RPI.23
- new net DEL_BLEU_3: LED102.A, LED124.A, LED125.A, LED126.A, LED127.A, LED128.A, LED129.A, LED130.A, T24.E
- new net DEL_BLEU_3_PWM: R81.2, RPI.13
- new net DEL_GYRO_1G: GYRO.1, R40.2
- new net DEL_GYRO_1_PWMG: R39.1, U$1.6
- new net DEL_GYRO_2G: GYRO.3, R42.2
- new net DEL_GYRO_2_PWMG: R41.1, U$1.20/A6
- new net DEL_JAUNE_1: LED132.A, LED149.A, LED150.A, LED151.A, LED152.A, LED153.A, LED154.A, LED155.A, T19.E
- new net DEL_JAUNE_1_PWM: R61.2, RPI.37
- new net DEL_JAUNE_2: LED34.A, LED51.A, LED52.A, LED53.A, LED54.A, LED55.A, LED56.A, LED57.A, T15.E
- new net DEL_JAUNE_2_PWM: R68.2, RPI.29
- new net DEL_JAUNE_3: LED100.A, LED117.A, LED118.A, LED119.A, LED120.A, LED121.A, LED122.A, LED123.A, T23.E
- new net DEL_JAUNE_3_PWM: R80.2, RPI.15
- new net DEL_ORANGE_1: LED131.A, LED135.A, LED136.A, LED137.A, LED138.A, LED139.A, LED140.A, LED141.A, T17.E
- new net DEL_ORANGE_1_PWM: R59.2, RPI.38
- new net DEL_ORANGE_2: LED33.A, LED37.A, LED38.A, LED39.A, LED40.A, LED41.A, LED42.A, LED43.A, T13.E
- new net DEL_ORANGE_2_PWM: R66.2, RPI.31
- new net DEL_ORANGE_3: LED103.A, LED104.A, LED105.A, LED106.A, LED107.A, LED108.A, LED109.A, LED99.A, T21.E
- new net DEL_ORANGE_3_PWM: R78.2, RPI.19
- new net DEL_POWER: DC7.3, T13.C, T14.C, T15.C, T16.C, T17.C, T18.C, T19.C, T20.C, T21.C, T22.C, T23.C, T24.C
- new net DEL_VERT_1: LED133.A, LED142.A, LED143.A, LED144.A, LED145.A, LED146.A, LED147.A, LED148.A, T18.E
- new net DEL_VERT_1_PWM: R60.2, RPI.40
- new net DEL_VERT_2: LED35.A, LED44.A, LED45.A, LED46.A, LED47.A, LED48.A, LED49.A, LED50.A, T14.E
- new net DEL_VERT_2_PWM: R67.2, RPI.33
- new net DEL_VERT_3: LED101.A, LED110.A, LED111.A, LED112.A, LED113.A, LED114.A, LED115.A, LED116.A, T22.E
- new net DEL_VERT_3_PWM: R79.2, RPI.21
- new net GNDB: C18.1, C19.1, C20.1, DC6.2, DC7.2, DEBUG_UART.1, LED97.K, LED98.K, LIPO1.1, LIPO1.2, R46.2, R47.2, R48.2, R49.2, R50.2, R51.2, R52.2, R53.2, R54.2, R55.2, R56.2, R57.2, R58.2, R63.2, R64.2, R65.2, R70.2, R71.2, R72.2, R73.2, R74.2, R75.2, R76.2, R77.2, RPI.14, RPI.20, RPI.25, RPI.30, RPI.34, RPI.39, RPI.6, RPI.9, U$4.3, U$4.4
- new net GNDG: AX12_G1.GND, C12.2, C13.2, C14.2, C15.2, C16.2, C17.2, DC-DC-6V.GND, DC5.2, GRUE1.3, GRUE1.4, GRUE1.5, GRUE1.6, GYRO.2, GYRO.4, H-BRIDGE1:C1.1, H-BRIDGE1:C2.1, H-BRIDGE1:D1.A, H-BRIDGE1:D4.A, H-BRIDGE1:D5.A, H-BRIDGE1:D8.A, H-BRIDGE1:IC1.1, H-BRIDGE1:IC1.15, H-BRIDGE1:IC1.8, H-BRIDGE1:R1.2, H-BRIDGE1:R2.2, H-BRIDGE1:R3.2, H-BRIDGE1:R4.2, H-BRIDGE1:R5.2, H-BRIDGE1:R6.2, IC1.1, MOT_H.3, MOT_V.3, MULTI-BUTTON-1:C1.1, MULTI-BUTTON-1:R2.2, MULTI-BUTTON-1:R3.2, MULTI-BUTTON-1:U3.3, MULTI-BUTTON-1:U3.4, MULTI-BUTTON-2:C1.1, MULTI-BUTTON-2:R2.2, MULTI-BUTTON-2:R3.2, MULTI-BUTTON-2:U3.3, MULTI-BUTTON-2:U3.4, R43.1, TOF_LP_D_AND_DISPLAY.1, TOF_LP_G.1, TOF_PINCE.1, U$1.AGND, U$1.GND, XL320_G1.GND, XL320_G2.GND
- new net GRUE_SERIAL_MISOG: GRUE1.2, U$1.1
- new net GRUE_SERIAL_MOSIG: GRUE1.1, U$1.0
- new net MOT_H_EN: H-BRIDGE1:IC1.6, H-BRIDGE1:R1.1, U$1.3
- new net MOT_H_ENC_A: MOT_H.5, U$1.11
- new net MOT_H_ENC_B: MOT_H.6, U$1.12
- new net MOT_H_IN1: H-BRIDGE1:IC1.5, H-BRIDGE1:R3.1, U$1.4
- new net MOT_H_IN2: H-BRIDGE1:IC1.7, H-BRIDGE1:R4.1, U$1.5
- new net MOT_H_OUT+: H-BRIDGE1:D1.C, H-BRIDGE1:D2.A, H-BRIDGE1:IC1.2, MOT_H.1
- new net MOT_H_OUT-: H-BRIDGE1:D3.A, H-BRIDGE1:D4.C, H-BRIDGE1:IC1.3, MOT_H.2
- new net MOT_V_EN: H-BRIDGE1:IC1.11, H-BRIDGE1:R2.1, U$1.21/A7
- new net MOT_V_ENC_A: MOT_V.5, U$1.15/A1
- new net MOT_V_ENC_B: MOT_V.6, U$1.16/A2
- new net MOT_V_IN1: H-BRIDGE1:IC1.10, H-BRIDGE1:R5.1, U$1.22/A8
- new net MOT_V_IN2: H-BRIDGE1:IC1.12, H-BRIDGE1:R6.1, U$1.23/A9
- new net MOT_V_OUT+: H-BRIDGE1:D5.C, H-BRIDGE1:D6.A, H-BRIDGE1:IC1.13, MOT_V.1
- new net MOT_V_OUT-: H-BRIDGE1:D7.A, H-BRIDGE1:D8.C, H-BRIDGE1:IC1.14, MOT_V.2
- new net MULTI-BUTTON-1:N$3: MULTI-BUTTON-1:R2.1, MULTI-BUTTON-1:U2.3, MULTI-BUTTON-1:U2.4
- new net MULTI-BUTTON-1:N$4: MULTI-BUTTON-1:R3.1, MULTI-BUTTON-1:U1.3, MULTI-BUTTON-1:U1.4
- new net MULTI-BUTTON-2:N$3: MULTI-BUTTON-2:R2.1, MULTI-BUTTON-2:U2.3, MULTI-BUTTON-2:U2.4
- new net MULTI-BUTTON-2:N$4: MULTI-BUTTON-2:R3.1, MULTI-BUTTON-2:U1.3, MULTI-BUTTON-2:U1.4
- new net N$19: R40.1, T11.E
- new net N$20: R39.2, T11.B
- new net N$23: R42.1, T12.E
- new net N$24: R41.2, T12.B
- new net N$27: DC-DC-6V.TRIM+, R43.2
- new net N$28: MULTI-BUTTON-1:C1.2, MULTI-BUTTON-1:R1.2, MULTI-BUTTON-1:U1.1, MULTI-BUTTON-1:U1.2, MULTI-BUTTON-1:U2.1, MULTI-BUTTON-1:U2.2, MULTI-BUTTON-1:U3.1, MULTI-BUTTON-1:U3.2, U$1.A10
- new net N$31: MULTI-BUTTON-2:C1.2, MULTI-BUTTON-2:R1.2, MULTI-BUTTON-2:U1.1, MULTI-BUTTON-2:U1.2, MULTI-BUTTON-2:U2.1, MULTI-BUTTON-2:U2.2, MULTI-BUTTON-2:U3.1, MULTI-BUTTON-2:U3.2, U$1.A11
- new net N$32: F1.1, H-BRIDGE1:C1.2, H-BRIDGE1:D2.C, H-BRIDGE1:D3.C, H-BRIDGE1:D6.C, H-BRIDGE1:D7.C, H-BRIDGE1:IC1.4
- new net N$35: F2.1, LIPO1.3, LIPO1.4
- new net N$36: D2.A, F2.2
- new net N$39: D2.C, S2.2
- new net N$40: LED97.A, R44.2
- new net N$43: LED98.A, R45.2
- new net N$44: LED33.K, LED37.K, LED38.K, LED39.K, R46.1
- new net N$47: LED40.K, LED41.K, LED42.K, LED43.K, R47.1
- new net N$48: LED35.K, LED44.K, LED45.K, LED46.K, R48.1
- new net N$51: LED47.K, LED48.K, LED49.K, LED50.K, R49.1
- new net N$52: LED34.K, LED51.K, LED52.K, LED53.K, R50.1
- new net N$55: LED131.K, LED135.K, LED136.K, LED137.K, R51.1
- new net N$56: LED138.K, LED139.K, LED140.K, LED141.K, R52.1
- new net N$57: LED133.K, LED142.K, LED143.K, LED144.K, R53.1
- new net N$58: LED145.K, LED146.K, LED147.K, LED148.K, R54.1
- new net N$59: LED132.K, LED149.K, LED150.K, LED151.K, R55.1
- new net N$60: LED152.K, LED153.K, LED154.K, LED155.K, R56.1
- new net N$61: LED134.K, LED156.K, LED157.K, LED158.K, R57.1
- new net N$62: LED159.K, LED160.K, LED161.K, LED162.K, R58.1
- new net N$63: R59.1, T17.B
- new net N$64: R60.1, T18.B
- new net N$65: R61.1, T19.B
- new net N$66: R62.1, T20.B
- new net N$67: LED54.K, LED55.K, LED56.K, LED57.K, R63.1
- new net N$68: LED36.K, LED58.K, LED59.K, LED60.K, R64.1
- new net N$69: LED61.K, LED62.K, LED63.K, LED64.K, R65.1
- new net N$70: R66.1, T13.B
- new net N$71: R67.1, T14.B
- new net N$72: R68.1, T15.B
- new net N$73: R69.1, T16.B
- new net N$74: LED103.K, LED104.K, LED105.K, LED99.K, R70.1
- new net N$75: LED106.K, LED107.K, LED108.K, LED109.K, R71.1
- new net N$76: LED101.K, LED110.K, LED111.K, LED112.K, R72.1
- new net N$77: LED113.K, LED114.K, LED115.K, LED116.K, R73.1
- new net N$78: LED100.K, LED117.K, LED118.K, LED119.K, R74.1
- new net N$79: LED120.K, LED121.K, LED122.K, LED123.K, R75.1
- new net N$80: LED102.K, LED124.K, LED125.K, LED126.K, R76.1
- new net N$81: LED127.K, LED128.K, LED129.K, LED130.K, R77.1
- new net N$82: R78.1, T21.B
- new net N$83: R79.1, T22.B
- new net N$84: R80.1, T23.B
- new net N$85: R81.1, T24.B
- new net POWEROFF: C20.2, R82.2, RPI.11, U$4.1, U$4.2
- new net RX: DEBUG_UART.4, RPI.10
- new net SCLG: TOF_LP_D_AND_DISPLAY.4, TOF_LP_G.4, TOF_PINCE.4, U$1.19/A5
- new net SDAG: TOF_LP_D_AND_DISPLAY.3, TOF_LP_G.3, TOF_PINCE.3, U$1.18/A4
- new net SERIAL_AX12G: Q3.2, R35.2, U$1.10, U$1.9
- new net SERIAL_AX12_5VG: AX12_G1.DATA, Q3.3, R36.2
- new net SERIAL_XL320G: Q4.2, R37.2, U$1.7, U$1.8
- new net SERIAL_XL320_5VG: Q4.3, R38.2, XL320_G1.DATA, XL320_G2.DATA
- new net STATUS_LED: R45.1, RPI.35
- new net TOF_LP_D: TOF_LP_D_AND_DISPLAY.5, U$1.13
- new net TOF_LP_G: TOF_LP_G.5, U$1.2
- new net TOF_PINCE_EXT: TOF_PINCE.6, U$1.17/A3
- new net TOF_PINCE_INT: TOF_PINCE.5, U$1.14/A0
- new net TX: DEBUG_UART.5, RPI.8
- new net VIN: U$1.VIN
- new net VUSB: U$1.VUSB
Routing:
- net DEL_POWER: track 0.00 -> 268.2 mm, vias 0 -> 12
- net +6V: track 0.00 -> 190.3 mm, vias 0 -> 2
- net DEL_VERT_3_PWM: track 0.00 -> 145.9 mm
- net +3V3G: track 0.00 -> 141.4 mm, vias 0 -> 9
- net DEL_ORANGE_3_PWM: track 0.00 -> 134.5 mm
- net DEL_BLEU_2: track 0.00 -> 130.8 mm, vias 0 -> 2
- net DEL_BLEU_3: track 0.00 -> 130.8 mm, vias 0 -> 2
- net DEL_BLEU_1: track 0.00 -> 130.8 mm, vias 0 -> 2
- net DEL_BLEU_3_PWM: track 0.00 -> 127.4 mm
- net DEL_JAUNE_3_PWM: track 0.00 -> 123.9 mm
- net +5VB: track 0.00 -> 109.2 mm
- net DEL_JAUNE_2: track 0.00 -> 107.7 mm
- net DEL_JAUNE_3: track 0.00 -> 107.7 mm
- net DEL_JAUNE_1: track 0.00 -> 107.7 mm
- net GNDB: track 0.00 -> 106.2 mm, vias 0 -> 7
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- added copper zone on layer 1, net GNDB
- added copper zone on layer 16, net GNDB
- added copper zone on layer 1, net GNDG
- added copper zone on layer 16, net GNDG
Other:
- board size 129 x 106 mm -> 196 x 160 mm
- board text added: "B"
- board text added: "GYRO"
- board text added: "O"
- board text added: "TOF LPD"
- board text added: "TOF LPG"
- board text added: "TOF PINCE"
- board text added: "V"
