File: electronique/intech-senpai-camion-grue-complet.sch (EAGLE design)
At the start: 95 parts, among them IC3 REG1117, P1 RGEF800, Q1 BSS138, Q2 BSS138, U1 TEENSY_3.5_DIL+USB, U2 TEENSY_3.1-3.2_DIL

Commit message: Elec version finale + Ajout fichiers gerber
Parts:
- added AX12_G1: DYNAMIXEL-1X03AX, 1NTech_pinhead:DYNAMIXEL-1X03AX
- added C12, C13, C17: 1µF, resistor:C-EUC0805
- added C14, C15, C18, C19, C20: 10µF, resistor:C-EUC0805
- added C16: 22µF, resistor:C-EUC0805
- added D2: S1M, diode:S1M
- added DC-DC-6V: DC-DC-CONVERTER, dc-dc-converter-6v:DC-DC-CONVERTER
- added DC5, DC7: R-78C3.3-1.0, dc-dc-converter:R-78C3.3-1.0
- added DC6: R-78C5.0-1.0, dc-dc-converter:R-78C5.0-1.0
- added DEBUG_UART, MOT_H, MOT_V: (no value), pinhead:PINHD-1X6
- added F1: MF-LSMF300, polyswitch:MF-LSMF300
- added F2: MF-MSMF110, polyswitch:MF-MSMF110
- added GRUE1: JST-10, con-jst:JST-10
- added GYRO, LIPO1: JST-04GH-V, con-jst:JST-04GH-V
- added IC1: REG1117, burr-brown:REG1117
- added LED100, LED117, LED118, LED119, LED120, LED121, LED122, LED123, LED132, LED149, LED150, LED151, LED152, LED153, LED154, LED155, LED34, LED51, LED52, LED53, LED54, LED55, LED56, LED57: jaune, led:LED5MM
- added LED101, LED110, LED111, LED112, LED113, LED114, LED115, LED116, LED133, LED142, LED143, LED144, LED145, LED146, LED147, LED148, LED35, LED44, LED45, LED46, LED47, LED48, LED49, LED50, LED97: vert, led:LED5MM
- added LED102, LED124, LED125, LED126, LED127, LED128, LED129, LED130, LED134, LED156, LED157, LED158, LED159, LED160, LED161, LED162, LED36, LED58, LED59, LED60, LED61, LED62, LED63, LED64, LED98: bleu, led:LED5MM
- added LED103, LED104, LED105, LED106, LED107, LED108, LED109, LED131, LED135, LED136, LED137, LED138, LED139, LED140, LED141, LED33, LED37, LED38, LED39, LED40, LED41, LED42, LED43, LED99: orange, led:LED5MM
- added Q3, Q4: BSS138, transistor-small-signal:BSS123
- added R35, R36, R37, R38: 10k, resistor:R-EU_R0805
- added R39, R41, R59, R60, R61, R62, R66, R67, R68, R69, R78, R79, R80, R81: 270, resistor:R-EU_R0805
- added R40, R42, R46, R47, R48, R49, R50, R51, R52, R53, R54, R55, R56, R57, R58, R63, R64, R65, R70, R71, R72, R73, R74, R75, R76, R77: 0, resistor:R-EU_R0805
- added R43: 220, resistor:R-EU_R0805
- added R44, R82: 1k, resistor:R-EU_R0805
- added R45: 470, resistor:R-EU_R0805
- added RPI: RPI-ZERO, RPI-Zero:RPI-ZERO
- added S2: TL36PO, switch:TL36PO
- added T11, T12, T13, T14, T15, T16, T17, T18, T19, T20, T21, T22, T23, T24: (no value), transistor:BC817-16-NPN-SOT23-BEC
- added TOF_LP_D_AND_DISPLAY, TOF_LP_G: JST-05, con-jst:JST-05
- added TOF_PINCE: JST-06, con-jst:JST-06
- added U$1: TEENSY_3.1-3.2_DIL+4, Teensy_libSG:TEENSY_3.1-3.2_DIL+4
- added U$4: PUSH-BUTTON, push-button:PUSH-BUTTON
- added XL320_G1, XL320_G2: DYNAMIXEL-1X03XL, 1NTech_pinhead:DYNAMIXEL-1X03XL
Connections:
- new net +12VB: C18.2, C19.2, DC6.VIN, DC7.VIN, S2.O
- new net +12VG: AX12_G1.DYN_VCC, C12.1, C14.1, C15.1, DC-DC-6V.VIN, DC5.VIN, GRUE1.10, GRUE1.7, GRUE1.8, GRUE1.9, IC1.VIN
- new net +3V3G: DC5.VOUT, Q3.G, Q4.G, R35.1, R37.1, T11.C, T12.C, TOF_LP_D_AND_DISPLAY.2, TOF_LP_G.2, TOF_PINCE.2, U$1.3.3V
- new net +5VB: DC6.VOUT, R44.1, RPI.5V0@1, RPI.5V0@2
- new net +5VG: C16.1, IC1.VOUT, MOT_H.4, MOT_V.4, R36.1, R38.1
- new net +6V: C13.1, C17.1, DC-DC-6V.VOUT, F1.2, XL320_G1.DYN_VCC, XL320_G2.DYN_VCC
- new net 3V3@1: R82.1, RPI.3V3@1
- new net ADC: C1.2, R1.2, U1.P$1, U2.P$1
- new net DEL_BLEU_1: LED134.A, LED156.A, LED157.A, LED158.A, LED159.A, LED160.A, LED161.A, LED162.A, T20.E
- new net DEL_BLEU_1_PWM: R62.2, RPI.GPIO16
- new net DEL_BLEU_2: LED36.A, LED58.A, LED59.A, LED60.A, LED61.A, LED62.A, LED63.A, LED64.A, T16.E
- new net DEL_BLEU_2_PWM: R69.2, RPI.GPIO11/SCLK
- new net DEL_BLEU_3: LED102.A, LED124.A, LED125.A, LED126.A, LED127.A, LED128.A, LED129.A, LED130.A, T24.E
- new net DEL_BLEU_3_PWM: R81.2, RPI.GPIO27/GEN2
- new net DEL_GYRO_1G: GYRO.1, R40.2
- new net DEL_GYRO_1_PWMG: R39.1, U$1.6/PWM
- new net DEL_GYRO_2G: GYRO.3, R42.2
- new net DEL_GYRO_2_PWMG: R41.1, U$1.20/A6/PWM
- new net DEL_JAUNE_1: LED132.A, LED149.A, LED150.A, LED151.A, LED152.A, LED153.A, LED154.A, LED155.A, T19.E
- new net DEL_JAUNE_1_PWM: R61.2, RPI.GPIO26
- new net DEL_JAUNE_2: LED34.A, LED51.A, LED52.A, LED53.A, LED54.A, LED55.A, LED56.A, LED57.A, T15.E
- new net DEL_JAUNE_2_PWM: R68.2, RPI.GPIO5
- new net DEL_JAUNE_3: LED100.A, LED117.A, LED118.A, LED119.A, LED120.A, LED121.A, LED122.A, LED123.A, T23.E
- new net DEL_JAUNE_3_PWM: R80.2, RPI.GPIO22/GEN3
- new net DEL_ORANGE_1: LED131.A, LED135.A, LED136.A, LED137.A, LED138.A, LED139.A, LED140.A, LED141.A, T17.E
- new net DEL_ORANGE_1_PWM: R59.2, RPI.GPIO20
- new net DEL_ORANGE_2: LED33.A, LED37.A, LED38.A, LED39.A, LED40.A, LED41.A, LED42.A, LED43.A, T13.E
- new net DEL_ORANGE_2_PWM: R66.2, RPI.GPIO6
- new net DEL_ORANGE_3: LED103.A, LED104.A, LED105.A, LED106.A, LED107.A, LED108.A, LED109.A, LED99.A, T21.E
- new net DEL_ORANGE_3_PWM: R78.2, RPI.GPIO10/MOSI
- new net DEL_POWER: DC7.VOUT, T13.C, T14.C, T15.C, T16.C, T17.C, T18.C, T19.C, T20.C, T21.C, T22.C, T23.C, T24.C
- new net DEL_VERT_1: LED133.A, LED142.A, LED143.A, LED144.A, LED145.A, LED146.A, LED147.A, LED148.A, T18.E
- new net DEL_VERT_1_PWM: R60.2, RPI.GPIO21
- new net DEL_VERT_2: LED35.A, LED44.A, LED45.A, LED46.A, LED47.A, LED48.A, LED49.A, LED50.A, T14.E
- new net DEL_VERT_2_PWM: R67.2, RPI.GPIO13
- new net DEL_VERT_3: LED101.A, LED110.A, LED111.A, LED112.A, LED113.A, LED114.A, LED115.A, LED116.A, T22.E
- new net DEL_VERT_3_PWM: R79.2, RPI.GPIO9/MISO
- new net ENABLE_A: IC1.ENABLE_A, R1.1
- new net ENABLE_B: IC1.ENABLE_B, R2.1
- new net GNDB: C18.1, C19.1, C20.1, DC6.GND, DC7.GND, DEBUG_UART.1, LED97.C, LED98.C, LIPO1.1, LIPO1.2, R46.2, R47.2, R48.2, R49.2, R50.2, R51.2, R52.2, R53.2, R54.2, R55.2, R56.2, R57.2, R58.2, R63.2, R64.2, R65.2, R70.2, R71.2, R72.2, R73.2, R74.2, R75.2, R76.2, R77.2, RPI.GND@1, RPI.GND@2, RPI.GND@3, RPI.GND@4, RPI.GND@5, RPI.GND@6, RPI.GND@7, RPI.GND@8, U$4.P$2
- new net GNDG: AX12_G1.GND, C12.2, C13.2, C14.2, C15.2, C16.2, C17.2, DC-DC-6V.GND, DC5.GND, GRUE1.3, GRUE1.4, GRUE1.5, GRUE1.6, GYRO.2, GYRO.4, IC1.GND, MOT_H.3, MOT_V.3, R43.1, TOF_LP_D_AND_DISPLAY.1, TOF_LP_G.1, TOF_PINCE.1, U$1.AGND, U$1.GND, XL320_G1.GND, XL320_G2.GND
- new net GRUE_SERIAL_MISOG: GRUE1.2, U$1.1/TX1/T
- new net GRUE_SERIAL_MOSIG: GRUE1.1, U$1.0/RX1/T
- new net INPUT3: IC1.INPUT3, R5.1
- new net INPUT4: IC1.INPUT4, R6.1
- new net LOGIC_HIGH: R1.1
- new net LOGIC_LOW: C1.1, R2.2, R3.2
- new net MOT_H_EN: U$1.3/CAN-TX/PWM
- new net MOT_H_ENC_A: MOT_H.5, U$1.11/MOSI
- new net MOT_H_ENC_B: MOT_H.6, U$1.12/MISO
- new net MOT_H_IN1: U$1.4/CAN-RX-PWM
- new net MOT_H_IN2: U$1.5/PWM
- new net MOT_H_OUT+: MOT_H.1
- new net MOT_H_OUT-: MOT_H.2
- new net MOT_V_EN: U$1.21/A7/PWM
- new net MOT_V_ENC_A: MOT_V.5, U$1.15/A1/T
- new net MOT_V_ENC_B: MOT_V.6, U$1.16/A2/T
- new net MOT_V_IN1: U$1.22/A8/T/PWM
- new net MOT_V_IN2: U$1.23/A9/T/PWM
- new net MOT_V_OUT+: MOT_V.1
- new net MOT_V_OUT-: MOT_V.2
- new net N$19: R40.1, T11.E
- new net N$20: R39.2, T11.B
- new net N$23: R42.1, T12.E
- new net N$24: R41.2, T12.B
- new net N$27: DC-DC-6V.TRIM+, R43.2
- new net N$28: U$1.A10
- new net N$31: U$1.A11
- new net N$32: F1.1
- new net N$35: F2.1, LIPO1.3, LIPO1.4
- new net N$36: D2.A, F2.2
- new net N$39: D2.C, S2.P
- new net N$40: LED97.A, R44.2
- new net N$43: LED98.A, R45.2
- new net N$44: LED33.C, LED37.C, LED38.C, LED39.C, R46.1
- new net N$47: LED40.C, LED41.C, LED42.C, LED43.C, R47.1
- new net N$48: LED35.C, LED44.C, LED45.C, LED46.C, R48.1
- new net N$51: LED47.C, LED48.C, LED49.C, LED50.C, R49.1
- new net N$52: LED34.C, LED51.C, LED52.C, LED53.C, R50.1
- new net N$55: LED131.C, LED135.C, LED136.C, LED137.C, R51.1
- new net N$56: LED138.C, LED139.C, LED140.C, LED141.C, R52.1
- new net N$57: LED133.C, LED142.C, LED143.C, LED144.C, R53.1
- new net N$58: LED145.C, LED146.C, LED147.C, LED148.C, R54.1
- new net N$59: LED132.C, LED149.C, LED150.C, LED151.C, R55.1
- new net N$60: LED152.C, LED153.C, LED154.C, LED155.C, R56.1
- new net N$61: LED134.C, LED156.C, LED157.C, LED158.C, R57.1
- new net N$62: LED159.C, LED160.C, LED161.C, LED162.C, R58.1
- new net N$63: R59.1, T17.B
- new net N$64: R60.1, T18.B
- new net N$65: R61.1, T19.B
- new net N$66: R62.1, T20.B
- new net N$67: LED54.C, LED55.C, LED56.C, LED57.C, R63.1
- new net N$68: LED36.C, LED58.C, LED59.C, LED60.C, R64.1
- new net N$69: LED61.C, LED62.C, LED63.C, LED64.C, R65.1
- new net N$70: R66.1, T13.B
- new net N$71: R67.1, T14.B
- new net N$72: R68.1, T15.B
- new net N$73: R69.1, T16.B
- new net N$74: LED103.C, LED104.C, LED105.C, LED99.C, R70.1
- new net N$75: LED106.C, LED107.C, LED108.C, LED109.C, R71.1
- new net N$76: LED101.C, LED110.C, LED111.C, LED112.C, R72.1
- new net N$77: LED113.C, LED114.C, LED115.C, LED116.C, R73.1
- new net N$78: LED100.C, LED117.C, LED118.C, LED119.C, R74.1
- new net N$79: LED120.C, LED121.C, LED122.C, LED123.C, R75.1
- new net N$80: LED102.C, LED124.C, LED125.C, LED126.C, R76.1
- new net N$81: LED127.C, LED128.C, LED129.C, LED130.C, R77.1
- new net N$82: R78.1, T21.B
- new net N$83: R79.1, T22.B
- new net N$84: R80.1, T23.B
- new net N$85: R81.1, T24.B
- new net OUT-: IC1.OUT2, IC1.OUT3
- new net OUT1: D1.C, D2.A, IC1.OUT1
- new net OUT2: IC1.OUT2
- new net OUT3: IC1.OUT3
- new net OUT4: IC1.OUT4
- new net POWEROFF: C20.2, R82.2, RPI.GPIO17/GEN0, U$4.P$1
- new net RX: DEBUG_UART.4, RPI.RXD0/GPIO15
- new net SCLG: TOF_LP_D_AND_DISPLAY.4, TOF_LP_G.4, TOF_PINCE.4, U$1.19/A5/T/SCL0
- new net SDAG: TOF_LP_D_AND_DISPLAY.3, TOF_LP_G.3, TOF_PINCE.3, U$1.18/A4/T/SDA0
- new net SERIAL_AX12G: Q3.S, R35.2, U$1.10/TX2/PWM, U$1.9/RX2/PWM
- new net SERIAL_AX12_5VG: AX12_G1.DATA, Q3.D, R36.2
- new net SERIAL_XL320G: Q4.S, R37.2, U$1.7/RX3, U$1.8/TX3
- new net SERIAL_XL320_5VG: Q4.D, R38.2, XL320_G1.DATA, XL320_G2.DATA
- new net STATUS_LED: R45.1, RPI.GPIO19
- new net TOF_LP_D: TOF_LP_D_AND_DISPLAY.5, U$1.13/SCK/LED
- new net TOF_LP_G: TOF_LP_G.5, U$1.2
- new net TOF_PINCE_EXT: TOF_PINCE.6, U$1.17/A3/T
- new net TOF_PINCE_INT: TOF_PINCE.5, U$1.14/A0
- new net TX: DEBUG_UART.5, RPI.TXD0/GPIO14
- net +12V: now also D2.C, IC1.VS
- net +5V: now also IC1.VCC
- net ENABLE: now also IC1.ENABLE_A, IC1.ENABLE_B
- net GND: now also IC1.GND, IC1.SEN_A, IC1.SEN_B, R4.2, R5.2, R6.2
- net INPUT1: now also IC1.INPUT1, IC1.INPUT4, R3.1
- net INPUT2: now also IC1.INPUT2, IC1.INPUT3, R4.1
- net N$3: now also R2.1, U2.P$2
- net N$4: now also R3.1, U1.P$2
- net OUT+: now also D2.A, IC1.OUT1, IC1.OUT4
